Commit message: Updated original urdf for first sander and made new urdf with new sander and mockup

File: crs_support/urdf/crs_v3.urdf (robot description, URDF)
Before this commit: robot crs, 16 links, 15 joints
Links:
- added link part; visual mesh filename=package://crs_support/meshes/Parts/visual/part1_ch.stl
- link eoat_link: geometry collision mesh filename=package://crs_support/meshes/end_effector/collision/ee_v2_c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; visual mesh filename=package://crs_support/meshes/end_effector/visual/ee_v2.stl
- link robot_stand: geometry collision box size=0.22 0.12 2.65; collision box size=0.22 0.12 2.65
Joints:
- added joint robot_stand_to_part_joint: type fixed, parent robot_stand, child part, origin xyz=-0.439 -1.1 -0.14 rpy=-3.1416 0.0 -1.571
- joint camera_optical_joint: origin xyz=0 0 0 rpy=-1.571 0 -1.571 -> xyz=-0.00345 0.070793 0.077409 rpy=-0.7854 0 0; parent gazebo_camera_link -> eoat_link
- joint gazebo_camera_joint: origin xyz=-0.04241 0.003917 0.0378 rpy=0 3.1416 0.0 -> xyz=0.0 0.0 0.0 rpy=1.57 -1.57 0.0; parent eoat_link -> camera_link_optical
- joint robot_base_joint: origin xyz=0.077 -2.019 1.020  rpy=0 1.571 0 -> xyz=0.036983 -2.0948 0.58  rpy=0 1.571 0
- joint sander_joint: origin xyz=0.10969 -0.001207 0.093395 rpy=0 1.571 0.0 -> xyz=0.0 -0.1167 0.12664 rpy=0.7854 0.0 0.0

Commit message: Updated to move part higher to reach more rasters

File: crs_support/urdf/crs_v3.urdf (robot description, URDF)
Before this commit: robot crs, 17 links, 16 joints
Joints:
- joint robot_stand_to_part_joint: origin xyz=-0.439 -1.1 -0.14 rpy=-3.1416 0.0 -1.571 -> xyz=-0.439 -1.2 -0.14 rpy=-3.1416 0.0 -1.571

Commit message: still getting memory leak

File: crs_support/urdf/crs_v3.urdf (robot description, URDF)
Before this commit: robot crs, 17 links, 16 joints
Joints:
- joint robot_stand_to_part_joint: origin xyz=-0.439 -1.2 -0.14 rpy=-3.1416 0.0 -1.571 -> xyz=-0.439 -1.1 -0.14 rpy=-3.1416 0.0 -1.571

Commit message: Updated joint limits to be more accurate

File: crs_support/urdf/crs_v3.urdf (robot description, URDF)
Before this commit: robot crs, 17 links, 16 joints
Joints:
- joint elbow_joint: limit lower=-2.6 upper=3.141592653589793 effort=150.0 velocity=3.14 -> lower=-6.28318530718 upper=6.28318530718 effort=150.0 velocity=3.14
