Commit message: Updated urdf to add FRAMOS and allow gazebo self-collisions

File: crs_support/urdf/swri_demo.urdf (robot description, URDF)
Before this commit: robot crs, 15 links, 14 joints
Links:
- link robot_stand: geometry collision box size=0.4318 0.4318 1.1; collision box size=0.889 0.889 0.7112
Joints:
- joint base_link-base_fixed_joint: origin xyz=0 0 0 rpy=-1.571 0 0 -> xyz=0 0 0 rpy=0 0 0
- joint robot_base_joint: axis 1 0 0 -> (none); origin xyz=0.077 -2.019 1.020  rpy=0 1.571 0 -> xyz=0 0 1.0922 rpy=0 0 0
- joint robot_stand_joint: origin xyz=0 0 0 rpy=-1.571 0 0 -> xyz=0 0 0 rpy=0 0 0

Commit message: Updated urdf

File: crs_support/urdf/swri_demo.urdf (robot description, URDF)
Before this commit: robot crs, 15 links, 14 joints
Links:
- added link part; visual mesh filename=package://crs_support/meshes/Parts/visual/part1_ch.stl
- added link sander_center_link
- link eoat_link: geometry collision mesh filename=package://crs_support/meshes/end_effector/collision/ee_v2_c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; visual mesh filename=package://crs_support/meshes/end_effector/visual/ee_v2.stl
- link robot_stand: geometry collision box size=0.22 0.12 2.65; collision box size=0.22 0.12 2.65
Joints:
- added joint robot_stand_to_part_joint: type fixed, parent robot_stand, child part, origin xyz=-0.439 -1.1 -0.14 rpy=-3.1416 0.0 -1.571
- added joint sander_joint: type fixed, parent eoat_link, child sander_center_link, origin xyz=0.0 -0.1167 0.12664 rpy=0.7854 0.0 0.0
- joint base_link-base_fixed_joint: origin xyz=0 0 0 rpy=0 0 0 -> xyz=0 0 0 rpy=-1.571 0 0
- joint camera_optical_joint: origin xyz=0 0 0 rpy=-1.571 0 -1.571 -> xyz=-0.00345 0.070793 0.077409 rpy=-0.7854 0 0; parent gazebo_camera_link -> eoat_link
- joint elbow_joint: limit lower=-2.6 upper=3.141592653589793 effort=150.0 velocity=3.14 -> lower=-6.28318530718 upper=6.28318530718 effort=150.0 velocity=3.14
- joint gazebo_camera_joint: origin xyz=0 0 0.02 rpy=0 0 1.571 -> xyz=0.0 0.0 0.0 rpy=1.57 -1.57 0.0; parent wrist_3_link -> camera_link_optical
- joint robot_base_joint: axis (none) -> 1 0 0; origin xyz=0 0 1.0922 rpy=0 0 0 -> xyz=0.036983 -2.0948 0.58  rpy=0 1.571 0
- joint robot_stand_joint: origin xyz=0 0 0 rpy=0 0 0 -> xyz=0 0 0 rpy=-1.571 0 0
- joint tool0_to_eoat_link: origin xyz=-0.04 0.09 -0.03 rpy=1.57 0.0 0 -> xyz=0.00 0.00 0.00 rpy=0.0 0.0 0
