Commit message: Modifications to test new motion execution in SWRI env

File: crs_support/urdf/swri_demo3.urdf.xacro (robot description, xacro)
@@ -22,6 +22,5 @@
     </link>
     <joint name="world_to_table_joint" type="fixed">
-<!--      <origin xyz="0 0 -0.363"/>-->
-      <origin xyz="0 0 -0.353"/>
+      <origin xyz="0 0 -0.363"/>
 <!--      <origin xyz="0 0 -0.385"/>-->
       <parent link="world"/>
@@ -55,4 +54,17 @@
     <link name="${prefix}external_walls">
       <visual>
+        <origin xyz="0 -1.2 -0.36"/>
+        <geometry>
+          <box size="$(arg table_size) 0.4 0.5"/>
+        </geometry>
+        <material name="StainlessSteel"/>
+      </visual>
+      <collision>
+        <origin xyz="0 -1.2 -0.36"/>
+        <geometry>
+          <box size="$(arg table_size) 0.4 0.5"/>
+        </geometry>
+      </collision>
+      <visual>
         <origin xyz="0 0.765 0"/>
         <geometry>
@@ -309,19 +321,6 @@
     </joint>
     <link name="${prefix}eoat_link">
-      <visual>
-          <geometry>
-              <mesh filename="package://crs_support/meshes/end_effector/visual/full_ee_v4.stl" />
-          </geometry>
-          <material name="Orange">
-              <color rgba="1.0 0.4 0.0 1.0" />
-          </material>
-      </visual>
-      <collision>
-          <geometry>
-              <mesh filename="package://crs_support/meshes/end_effector/collision/full_ee_v4_collision.stl" />
-          </geometry>
-      </collision>
-<!--      <inertial>
-        <origin xyz="8.625E-08 -4.6583E-06 0.03145" rpy="0 0 0" />
+      <inertial>
+<!--        <origin xyz="8.625E-08 -4.6583E-06 0.03145" rpy="0 0 0" />-->
         <origin xyz="0 0 0" rpy="0 0 0" />
         <mass value="0.22652" />
@@ -360,141 +359,20 @@
           <mesh filename="package://crs_support/meshes/end_effector/visual/ee1.stl" />
         </geometry>
-      </collision>-->
+      </collision>
     </link>
     <joint name="${prefix}tool0_to_eoat_link" type="fixed">
         <parent link="${prefix}tool0" />
         <child link="${prefix}eoat_link" />
-<!--        <origin xyz="0 0 0" rpy="1.57 0 -1.57" />-->
-        <origin xyz="0 0 0" rpy="0 0 0" />
-    </joint>
-    <link name="${prefix}robot_stand">
-        <visual>
-            <geometry>
-                <box size="0.4318 0.4318 1.1"/>
-            </geometry>
-            <material name="LightGrey">
-                <color rgba="0.7 0.7 0.7 1.0" />
-            </material>
-            <origin rpy="0 0 0" xyz="0 0 0.55" />
-        </visual>
-        <visual>
-            <geometry>
-                <box size="0.889 0.889 0.7112"/>
-            </geometry>
-            <material name="LightGrey">
-                <color rgba="0.7 0.7 0.7 1.0" />
-            </material>
-            <origin rpy="0 0 0" xyz="0 0 0.3556" />
-        </visual>
-        <visual>
-            <geometry>
-                <box size="1.55 1.55 0.254"/>
-            </geometry>
-            <material name="LightGrey">
-                <color rgba="0.7 0.7 0.7 1.0" />
-            </material>
-            <origin rpy="0 0 0" xyz="0 0 0.127" />
-        </visual>
-        <visual>
-            <geometry>
-                <box size="1.55 1.55 1.1"/>
-            </geometry>
-            <material name="Green">
-                <color rgba="0.0 0.5 0.0 1.0" />
-            </material>
-            <origin rpy="0 0 0" xyz="0 1 0.55" />
-        </visual>
-        <collision>
-            <geometry>
-                <box size="0.4318 0.4318 1.1"/>
-            </geometry>
-            <material name="LightGrey">
-                <color rgba="0.7 0.7 0.7 1.0" />
-            </material>
-            <origin rpy="0 0 0" xyz="0 0 0.55" />
-        </collision>
-        <collision>
-            <geometry>
-                <box size="0.889 0.889 0.7112"/>
-            </geometry>
-            <material name="LightGrey">
-                <color rgba="0.7 0.7 0.7 1.0" />
-            </material>
-            <origin rpy="0 0 0" xyz="0 0 0.3556" />
-        </collision>
-        <collision>
-            <geometry>
-                <box size="1.55 1.55 0.254"/>
-            </geometry>
-            <material name="LightGrey">
-                <color rgba="0.7 0.7 0.7 1.0" />
-            </material>
-            <origin rpy="0 0 0" xyz="0 0 0.127" />
-        </collision>
-        <collision>
-            <geometry>
-                <box size="1.55 1.55 1.1"/>
-            </geometry>
-            <material name="Green">
-                <color rgba="0.0 0.5 0.0 1.0" />
-            </material>
-            <origin rpy="0 0 0" xyz="0 1 0.55" />
-        </collision>
-        <inertial>
-            <mass value="0.1" />
-            <inertia ixx="0.03" iyy="0.03" izz="0.03" ixy="0.0" ixz="0.0" iyz="0.0" />
-        </inertial>
+        <origin xyz="0 0 0" rpy="1.57 0 -1.57" />
+    </joint>
     <link name="${prefix}sander_center_link" />
-    <link name="${prefix}sander_intermediate_link">
-      <visual>
-          <geometry>
-              <cylinder length="0.025" radius="0.06425" />
-          </geometry>
-          <origin rpy="0 0 0" xyz="0 0 0" />
-      </visual>
-      <collision>
-          <geometry>
-              <cylinder length="0.025" radius="0.06425" />
-          </geometry>
-          <origin rpy="0 0 0" xyz="0 0 0" />
-      </collision>
-    </link>
-    <joint name="${prefix}sander_intermediate_to_sander_center_link" type="fixed">
-      <parent link="${prefix}sander_intermediate_link" />
-      <child link="${prefix}sander_center_link" />
+    <joint name="${prefix}tool0_to_sander_center_link" type="fixed">
+        <parent link="${prefix}eoat_link" />
+        <child link="${prefix}sander_center_link" />
 <!--        <origin xyz="0 0.16578 0.01902" rpy="-0.785 0 0" />-->
-<!--        <origin xyz="0 0.162 0.015" rpy="-0.785 0 0" />-->
+        <origin xyz="0 0.162 0.015" rpy="-0.785 0 0" />
 <!--        <origin xyz="0 0.04612 -0.03371" rpy="-2.355 0 0" />-->
-      <origin  xyz="0.0 0.0 0.0125" rpy="0.0 0.0 0.0"/>
-    </joint>
-    <joint name="${prefix}tool0_to_sander_intermediate_link" type="fixed">
-        <parent link="${prefix}eoat_link" />
-        <child link="${prefix}sander_intermediate_link" />
-<!--        <origin xyz="0 0.16578 0.01902" rpy="-0.785 0 0" />-->
-<!--        <origin xyz="0 0.162 0.015" rpy="-0.785 0 0" />-->
-<!--        <origin xyz="0 0.04612 -0.03371" rpy="-2.355 0 0" />-->
-        <origin xyz="0.0 -0.15497 0.17503" rpy="0.7854 0.0 0.0"/>
-    </joint>
-    <link name="${prefix}gazebo_camera_link" />
-    <joint name="${prefix}gazebo_camera_joint" type="fixed">
-        <origin xyz="0.0 0.0 0.0" rpy="1.57 -1.57 0.0"/>
-        <parent link="${prefix}camera_link_optical"/>
-        <child link="${prefix}gazebo_camera_link"/>
-    </joint>
-    <link name="${prefix}camera_link_optical" />
-    <joint name="${prefix}camera_optical_joint" type="fixed">
-        <origin xyz="-0.00345 0.070793 0.077409" rpy="-0.7854 0 0"/>
-        <parent link="${prefix}eoat_link"/>
-        <!-- <parent link="${prefix}gazebo_camera_link"/> -->
-        <child link="${prefix}camera_link_optical"/>
-    </joint>
-    <link name="${prefix}camera_link" />
-    <joint name="${prefix}camera_link_joint" type="fixed">
-<!--        <origin xyz="0.001 0.015 0.0" rpy="-1.57 1.57 0"/>-->
-        <origin xyz="0.0 0.0 0.0" rpy="1.57 -1.57 0"/>
-        <parent link="${prefix}camera_link_optical"/>
-        <child link="${prefix}camera_link"/>
-    </joint>
-    <link name="${prefix}part" >
+    </joint>
+<!--    <link name="${prefix}part" >
         <visual>
             <geometry>
@@ -506,5 +384,5 @@
             <origin rpy="0 0 0" xyz="0 0 -0.25" />
         </visual>
-<!--        <visual>
+        <visual>
             <origin rpy="0 0 0" xyz="0 0 0" />
             <geometry>
@@ -519,12 +397,12 @@
                 <mesh filename="package://crs_support/meshes/Parts/collision/part1_ch.stl" />
             </geometry>
-        </collision>-->
-    </link>
-    <joint name="${prefix}robot_stand_to_part_joint" type= "fixed">
-<!--        <origin xyz="-0.5 0.5 1.3" rpy= "1.571 -1.571 0"/>-->
-        <origin xyz="-0.25 0.5 1.15" rpy= "0.0 0.0 0"/>
-        <parent link="${prefix}robot_stand"/>
+        </collision>
+    </link>-->
+<!--    <joint name="${prefix}robot_stand_to_part_joint" type= "fixed">
+        <origin xyz="-0.5 0.5 1.3" rpy= "1.571 -1.571 0"/>
+        <origin xyz="0.25 -0.28 0.0" rpy= "0.0 0.0 1.571"/>
+        <parent link="table"/>
         <child link="${prefix}part"/>
-    </joint>
+    </joint>-->
     <transmission name="trans_shoulder_pan_joint">
         <type>transmission_interface/SimpleTransmission</type>
@@ -660,12 +538,12 @@
             <ros>
               <namespace>custom_ns</namespace>
-              <argument>camera/image_raw:=camera/custom_image</argument>
-              <argument>camera/image_depth:=camera/custom_image_depth</argument>
-              <argument>camera/camera_info:=camera/custom_info_raw</argument>
-              <argument>camera/camera_info_depth:=camera/custom_info_depth</argument>
-              <argument>camera/points:=camera/pointcloud</argument>
+              <argument>custom_camera/image_raw:=custom_camera/custom_image</argument>
+              <argument>custom_camera/image_depth:=custom_camera/custom_image_depth</argument>
+              <argument>custom_camera/camera_info:=custom_camera/custom_info_raw</argument>
+              <argument>custom_camera/camera_info_depth:=custom_camera/custom_info_depth</argument>
+              <argument>custom_camera/points:=custom_camera/custom_points</argument>
             </ros>
             <!-- Set camera name. If empty, defaults to sensor name (i.e. "sensor_name") -->
-            <camera_name>camera</camera_name>
+            <camera_name>custom_camera</camera_name>
             <frame_name>camera_link_optical</frame_name>
             <!-- Set TF frame name. If empty, defaults to link name (i.e. "link_name") -->
