Commit message: Updated swri urdf envrionment

File: crs_support/urdf/swri_demo2.urdf.xacro (robot description, xacro)
@@ -2,6 +2,8 @@
 <robot name="crs" xmlns:xacro="http://ros.org/wiki/xacro">
   <xacro:macro name="crs_workcell" params="prefix:=^|''">
-  <xacro:arg name="table_size" default="3.0"/>
-    <link name="world"/>
+  <xacro:arg name="table_size" default="1.5"/>
+  <xacro:property name="BASE_PLATE_THICKNESS" value="0.00635" scope="parent"/>
+  <xacro:property name="BASE_PLATE_LENGTH" value="0.762" scope="parent"/>
+  <xacro:property name="BASE_PLATE_WIDTH" value="0.3048" scope="parent"/>
     <link name="table">
       <visual>
@@ -22,53 +24,55 @@
     </link>
     <joint name="world_to_table_joint" type="fixed">
-<!--      <origin xyz="0 0 -0.363"/>-->
-      <origin xyz="0 0 -0.353"/>
-<!--      <origin xyz="0 0 -0.385"/>-->
+      <origin xyz="0 0 1.0"/>
       <parent link="world"/>
       <child link="table"/>
     </joint>
-  <!--  <link name="${prefix}part"/>
-    <joint name="table_to_part" type="fixed">
-      <origin xyz="0.0 -0.875 -0.008" />
-      <parent link="table"/>
-      <child link="${prefix}part"/>
-    </joint>-->
-    <link name="robot_stand">
+    <link name="base_plate">
       <visual>
-        <origin xyz="0 0 -0.1905"/>
+        <origin xyz="${0.5 * BASE_PLATE_WIDTH} ${0.5 * BASE_PLATE_LENGTH} ${BASE_PLATE_THICKNESS}"/>
         <geometry>
-          <box size="0.35 0.35 0.381"/>
+          <box size="${BASE_PLATE_WIDTH} ${BASE_PLATE_LENGTH} ${BASE_PLATE_THICKNESS}"/>
         </geometry>
+        <material name="StainlessSteel">
+          <color rgba="0.6 0.6 0.6 1.0"/>
+        </material>
       </visual>
       <collision>
-        <origin xyz="0 0 -0.1905"/>
+        <origin xyz="${0.5 * BASE_PLATE_WIDTH} ${0.5 * BASE_PLATE_LENGTH} ${BASE_PLATE_THICKNESS}"/>
         <geometry>
-          <box size="0.35 0.35 0.381"/>
+          <box size="${BASE_PLATE_WIDTH} ${BASE_PLATE_LENGTH} ${BASE_PLATE_THICKNESS}"/>
+        </geometry>
+        <material name="StainlessSteel">
+          <color rgba="0.6 0.6 0.6 1.0"/>
+        </material>
+      </collision>
+    </link>
+    <joint name="table_to_base_plate" type="fixed">
+      <origin xyz="${-0.5*$(arg table_size) + 0.1397 } ${-0.5*$(arg table_size) + 0.09525} 0.0" rpy="0 0 0"/>
+       <parent link="table"/>
+       <child link="base_plate"/>
+    </joint>
+    <!-- mold -->
+    <link name="layup_mold">
+      <visual>
+        <origin xyz="0 0 0" rpy="0 0 0"/>
+        <geometry>
+         <mesh filename="package://crs_support/meshes/Swri_demo/mold_transformed.stl"/>
+        </geometry>
+        <material name="white">
+          <color rgba="1 1 1 1"/>
+        </material>
+      </visual>
+      <collision>
+        <origin xyz="0 0 0"/>
+        <geometry>
+          <mesh filename="package://crs_support/meshes/Swri_demo/mold_transformed.stl"/>
         </geometry>
       </collision>
     </link>
-    <joint name="table_to_robot_stand" type="fixed">
-      <origin xyz="0.0 0.0 0.0" rpy="0.0 0.0 3.1415"/>
-      <parent link="world"/>
-      <child link="robot_stand"/>
-    </joint>
-    <link name="${prefix}external_walls">
-      <visual>
-        <origin xyz="0 0.765 0"/>
-        <geometry>
-          <box size="$(arg table_size) 0.1 $(arg table_size)"/>
-        </geometry>
-      </visual>
-      <collision>
-        <origin xyz="0 0.765 0"/>
-        <geometry>
-          <box size="$(arg table_size) 0.1 $(arg table_size)"/>
-        </geometry>
-      </collision>
-    </link>
-    <joint name="table_to_external_walls" type="fixed">
-      <origin xyz="0.0 0.0 0.0" rpy="0.0 0.0 0.0"/>
-      <parent link="world"/>
-      <child link="${prefix}external_walls"/>
+    <joint name="table_to_mold" type="fixed">
+      <parent link="table"/>
+      <child link="layup_mold"/>
+      <origin xyz="-0.30359 -0.13389 0.05497" rpy="-0.0091 -0.013 0.0197"/>
     </joint>
     <link name="${prefix}base_link">
@@ -292,9 +296,4 @@
     </link>
     <link name="${prefix}base" />
-    <joint name="table_to_ur" type="fixed">
-      <origin xyz="0.0 0.0 0.0" rpy="0.0 0.0 3.1415"/>
-      <parent link="world"/>
-      <child link="${prefix}base"/>
-    </joint>
     <joint name="${prefix}base_link-base_fixed_joint" type="fixed">
         <origin rpy="0 0 0" xyz="0 0 0" />
@@ -309,65 +308,51 @@
     </joint>
     <link name="${prefix}eoat_link">
-      <visual>
-          <geometry>
-              <mesh filename="package://crs_support/meshes/end_effector/visual/full_ee_v4.stl" />
-          </geometry>
-          <material name="Orange">
-              <color rgba="1.0 0.4 0.0 1.0" />
-          </material>
-      </visual>
-      <collision>
-          <geometry>
-              <mesh filename="package://crs_support/meshes/end_effector/collision/full_ee_v4_collision.stl" />
-          </geometry>
-      </collision>
-<!--      <inertial>
-        <origin xyz="8.625E-08 -4.6583E-06 0.03145" rpy="0 0 0" />
-        <origin xyz="0 0 0" rpy="0 0 0" />
-        <mass value="0.22652" />
-        <inertia ixx="0.00020005" ixy="-4.2442E-10" ixz="-2.9069E-10" iyy="0.00017832" iyz="-3.4402E-08" izz="0.00013478" />
-      </inertial>
-      <visual>
-        <origin xyz="0 0 0" rpy="0 0 0" />
-        <geometry>
-          <mesh filename="package://crs_support/meshes/end_effector/visual/ee1.stl" />
-        </geometry>
-        <material name="">
-          <color rgba="0.1 0.1 0.1 1" />
-        </material>
-      </visual>
-      <visual>
-        <origin xyz="0 0 0" rpy="0 0 0" />
-        <geometry>
-          <mesh filename="package://crs_support/meshes/end_effector/visual/ee2.stl" />
-        </geometry>
-        <material name="">
-          <color rgba="0.1 0.1 0.1 1" />
-        </material>
-      </visual>
-      <visual>
-        <origin xyz="0 0 0" rpy="0 0 0" />
-        <geometry>
-          <mesh filename="package://crs_support/meshes/end_effector/visual/ee3.stl" />
-        </geometry>
-        <material name="">
-          <color rgba="0.1 0.1 0.1 1" />
-        </material>
-      </visual>
-      <collision>
-        <origin xyz="0 0 0" rpy="0 0 0" />
-        <geometry>
-          <mesh filename="package://crs_support/meshes/end_effector/visual/ee1.stl" />
-        </geometry>
-      </collision>-->
+        <inertial>
+            <origin xyz="8.625E-08 -4.6583E-06 0.03145" rpy="0 0 0" />
+            <mass value="0.22652" />
+            <inertia ixx="0.00020005" ixy="-4.2442E-10" ixz="-2.9069E-10" iyy="0.00017832" iyz="-3.4402E-08" izz="0.00013478" />
+        </inertial>
+        <visual>
+            <origin xyz="0 0 0" rpy="0 0 0" />
+            <geometry>
+                <mesh filename="package://crs_support/meshes/Swri_demo/robotiq_2f_85_gripper_visualization/collision/robotiq_arg2f_base_link.stl" />
+<!--                <mesh filename="package://crs_support/meshes/Swri_demo/robotiq_2f_85_gripper_visualization/visual/robotiq_arg2f_85_base_link.dae" scale="0.001 0.001 0.001"/>-->
+            </geometry>
+            <material name="">
+                <color rgba="0.1 0.1 0.1 1" />
+            </material>
+        </visual>
+        <collision>
+            <origin xyz="0 0 0" rpy="0 0 0" />
+            <geometry>
+                <mesh filename="package://crs_support/meshes/Swri_demo/robotiq_2f_85_gripper_visualization/collision/robotiq_arg2f_base_link.stl" />
+            </geometry>
+        </collision>
+        <visual>
+            <geometry>
+                <cylinder radius="0.015" length="0.175"/>
+            </geometry>
+            <origin rpy="0 0 0" xyz="0 0 0.0875" />
+            <material name="">
+                <color rgba="0.1 0.1 0.1 1" />
+            </material>
+        </visual>
+        <collision>
+            <geometry>
+                <cylinder radius="0.015" length="0.175"/>
+            </geometry>
+            <origin rpy="0 0 0" xyz="0 0 0.0875" />
+            <material name="">
+                <color rgba="0.1 0.1 0.1 1" />
+            </material>
+        </collision>
     </link>
     <joint name="${prefix}tool0_to_eoat_link" type="fixed">
         <parent link="${prefix}tool0" />
         <child link="${prefix}eoat_link" />
-<!--        <origin xyz="0 0 0" rpy="1.57 0 -1.57" />-->
-        <origin xyz="0 0 0" rpy="0 0 0" />
+        <origin rpy="0.0 0.0 0" xyz="0.00 0.00 0.00" />
     </joint>
     <link name="${prefix}robot_stand">
-        <visual>
+<!--        <visual>
             <geometry>
                 <box size="0.4318 0.4318 1.1"/>
@@ -444,35 +429,20 @@
             <mass value="0.1" />
             <inertia ixx="0.03" iyy="0.03" izz="0.03" ixy="0.0" ixz="0.0" iyz="0.0" />
-        </inertial>
-    <link name="${prefix}sander_center_link" />
-    <link name="${prefix}sander_intermediate_link">
-      <visual>
-          <geometry>
-              <cylinder length="0.025" radius="0.06425" />
-          </geometry>
-          <origin rpy="0 0 0" xyz="0 0 0" />
-      </visual>
-      <collision>
-          <geometry>
-              <cylinder length="0.025" radius="0.06425" />
-          </geometry>
-          <origin rpy="0 0 0" xyz="0 0 0" />
-      </collision>
-    </link>
-    <joint name="${prefix}sander_intermediate_to_sander_center_link" type="fixed">
-      <parent link="${prefix}sander_intermediate_link" />
-      <child link="${prefix}sander_center_link" />
-<!--        <origin xyz="0 0.16578 0.01902" rpy="-0.785 0 0" />-->
-<!--        <origin xyz="0 0.162 0.015" rpy="-0.785 0 0" />-->
-<!--        <origin xyz="0 0.04612 -0.03371" rpy="-2.355 0 0" />-->
-      <origin  xyz="0.0 0.0 0.0125" rpy="0.0 0.0 0.0"/>
-    </joint>
-    <joint name="${prefix}tool0_to_sander_intermediate_link" type="fixed">
-        <parent link="${prefix}eoat_link" />
-        <child link="${prefix}sander_intermediate_link" />
-<!--        <origin xyz="0 0.16578 0.01902" rpy="-0.785 0 0" />-->
-<!--        <origin xyz="0 0.162 0.015" rpy="-0.785 0 0" />-->
-<!--        <origin xyz="0 0.04612 -0.03371" rpy="-2.355 0 0" />-->
-        <origin xyz="0.0 -0.15497 0.17503" rpy="0.7854 0.0 0.0"/>
+        </inertial>-->
+    </link>
+    <joint name="${prefix}robot_base_joint" type="fixed">
+        <!--<parent link="robot_stand" />
+        <child link="base" />
+        <origin rpy="0 0 0" xyz="0 0 1.0922" />-->
+        <parent link="layup_mold" />
+        <child link="base" />
+        <origin xyz="0.9545 0.0144 0.0797" rpy="0.0 0.0 3.1415"/>
+        <limit effort="1.0" lower="-0.1" upper="1.9" velocity=".01" />
+    </joint>
+    <link name="world" />
+    <joint name="${prefix}robot_stand_joint" type="fixed">
+        <parent link="world" />
+        <child link="${prefix}robot_stand" />
+        <origin rpy="0 0 0" xyz="0 0 0" />
     </joint>
     <link name="${prefix}gazebo_camera_link" />
@@ -489,10 +459,10 @@
         <child link="${prefix}camera_link_optical"/>
     </joint>
-    <link name="${prefix}camera_link" />
-    <joint name="${prefix}camera_link_joint" type="fixed">
-<!--        <origin xyz="0.001 0.015 0.0" rpy="-1.57 1.57 0"/>-->
-        <origin xyz="0.0 0.0 0.0" rpy="1.57 -1.57 0"/>
-        <parent link="${prefix}camera_link_optical"/>
-        <child link="${prefix}camera_link"/>
+    <link name="${prefix}sander_center_link" />
+    <joint name="${prefix}sander_joint" type = "fixed">
+<!--        <origin xyz="0.0 -0.15497 0.17503" rpy="0.7854 0.0 0.0"/>-->
+        <origin xyz="0.0 0.0 0.175" rpy="0.0 0.0 0.0"/>
+        <parent link="${prefix}eoat_link"/>
+        <child link="${prefix}sander_center_link" />
     </joint>
     <link name="${prefix}part" >
@@ -523,6 +493,6 @@
     <joint name="${prefix}robot_stand_to_part_joint" type= "fixed">
 <!--        <origin xyz="-0.5 0.5 1.3" rpy= "1.571 -1.571 0"/>-->
-        <origin xyz="-0.25 0.5 1.15" rpy= "0.0 0.0 0"/>
-        <parent link="${prefix}robot_stand"/>
+        <origin xyz="0.15 -0.5 0.0" rpy= "0.0 0.0 0"/>
+        <parent link="table"/>
         <child link="${prefix}part"/>
     </joint>
@@ -660,12 +630,12 @@
             <ros>
               <namespace>custom_ns</namespace>
-              <argument>camera/image_raw:=camera/custom_image</argument>
-              <argument>camera/image_depth:=camera/custom_image_depth</argument>
-              <argument>camera/camera_info:=camera/custom_info_raw</argument>
-              <argument>camera/camera_info_depth:=camera/custom_info_depth</argument>
-              <argument>camera/points:=camera/pointcloud</argument>
+              <argument>custom_camera/image_raw:=custom_camera/custom_image</argument>
+              <argument>custom_camera/image_depth:=custom_camera/custom_image_depth</argument>
+              <argument>custom_camera/camera_info:=custom_camera/custom_info_raw</argument>
+              <argument>custom_camera/camera_info_depth:=custom_camera/custom_info_depth</argument>
+              <argument>custom_camera/points:=custom_camera/custom_points</argument>
             </ros>
             <!-- Set camera name. If empty, defaults to sensor name (i.e. "sensor_name") -->
-            <camera_name>camera</camera_name>
+            <camera_name>custom_camera</camera_name>
             <frame_name>camera_link_optical</frame_name>
             <!-- Set TF frame name. If empty, defaults to link name (i.e. "link_name") -->

Commit message: Setup process planner test to test with surface executer

File: crs_support/urdf/swri_demo2.urdf.xacro (robot description, xacro)
@@ -3,5 +3,6 @@
   <xacro:macro name="crs_workcell" params="prefix:=^|''">
   <xacro:arg name="table_size" default="1.5"/>
-  <xacro:property name="BASE_PLATE_THICKNESS" value="0.6096" scope="parent"/> CHANGED TO ACCOUNT FOR KUKA
+<!--  <xacro:property name="BASE_PLATE_THICKNESS" value="0.6096" scope="parent"/> CHANGED TO ACCOUNT FOR KUKA-->
+  <xacro:property name="BASE_PLATE_THICKNESS" value="0.01" scope="parent"/> CHANGED TO ACCOUNT FOR KUKA
   <xacro:property name="BASE_PLATE_LENGTH" value="0.762" scope="parent"/>
   <xacro:property name="BASE_PLATE_WIDTH" value="0.3048" scope="parent"/>
@@ -16,10 +17,10 @@
         </material>
       </visual>
-      <collision>
+<!--      <collision>
         <origin xyz="0 0 -0.05"/>
         <geometry>
           <box size="$(arg table_size) $(arg table_size) 0.1"/>
         </geometry>
-      </collision>
+      </collision>-->
     </link>
     <joint name="world_to_table_joint" type="fixed">
@@ -64,10 +65,10 @@
         </material>
       </visual>
-      <collision>
+<!--      <collision>
         <origin xyz="0 0 0"/>
         <geometry>
           <mesh filename="package://crs_support/meshes/Swri_demo/mold_transformed.stl"/>
         </geometry>
-      </collision>
+      </collision>-->
     </link>
     <joint name="table_to_mold" type="fixed">
@@ -95,5 +96,5 @@
         </geometry>
       </visual>
-      <collision> Small square base plate
+<!--      <collision> Small square base plate
         <origin xyz="0.2286 -0.127 0.005" rpy="0 0 0"/>
         <geometry>
@@ -112,5 +113,5 @@
           <box size="0.7747 0.1143 0.0508"/>
         </geometry>
-      </collision>
+      </collision>-->
     </link>
     <joint name="table_to_table_obstacles" type="fixed">
