Commit message: code clean up, removed extra files

File: crs_support/urdf/swri_demo.urdf.xacro (robot description, xacro)
@@ -54,4 +54,17 @@
     </joint>
     <link name="${prefix}external_walls">
+      <visual>
+        <origin xyz="0 -1.2 -0.36"/>
+        <geometry>
+          <box size="$(arg table_size) 0.4 0.5"/>
+        </geometry>
+        <material name="StainlessSteel"/>
+      </visual>
+      <collision>
+        <origin xyz="0 -1.2 -0.36"/>
+        <geometry>
+          <box size="$(arg table_size) 0.4 0.5"/>
+        </geometry>
+      </collision>
       <visual>
         <origin xyz="0 0.765 0"/>
@@ -368,107 +381,8 @@
         <origin xyz="0 0 0" rpy="0 0 0" />
     </joint>
-    <link name="${prefix}robot_stand">
-        <visual>
-            <geometry>
-                <box size="0.4318 0.4318 1.1"/>
-            </geometry>
-            <material name="LightGrey">
-                <color rgba="0.7 0.7 0.7 1.0" />
-            </material>
-            <origin rpy="0 0 0" xyz="0 0 0.55" />
-        </visual>
-        <visual>
-            <geometry>
-                <box size="0.889 0.889 0.7112"/>
-            </geometry>
-            <material name="LightGrey">
-                <color rgba="0.7 0.7 0.7 1.0" />
-            </material>
-            <origin rpy="0 0 0" xyz="0 0 0.3556" />
-        </visual>
-        <visual>
-            <geometry>
-                <box size="1.55 1.55 0.254"/>
-            </geometry>
-            <material name="LightGrey">
-                <color rgba="0.7 0.7 0.7 1.0" />
-            </material>
-            <origin rpy="0 0 0" xyz="0 0 0.127" />
-        </visual>
-        <visual>
-            <geometry>
-                <box size="1.55 1.55 1.1"/>
-            </geometry>
-            <material name="Green">
-                <color rgba="0.0 0.5 0.0 1.0" />
-            </material>
-            <origin rpy="0 0 0" xyz="0 1 0.55" />
-        </visual>
-        <collision>
-            <geometry>
-                <box size="0.4318 0.4318 1.1"/>
-            </geometry>
-            <material name="LightGrey">
-                <color rgba="0.7 0.7 0.7 1.0" />
-            </material>
-            <origin rpy="0 0 0" xyz="0 0 0.55" />
-        </collision>
-        <collision>
-            <geometry>
-                <box size="0.889 0.889 0.7112"/>
-            </geometry>
-            <material name="LightGrey">
-                <color rgba="0.7 0.7 0.7 1.0" />
-            </material>
-            <origin rpy="0 0 0" xyz="0 0 0.3556" />
-        </collision>
-        <collision>
-            <geometry>
-                <box size="1.55 1.55 0.254"/>
-            </geometry>
-            <material name="LightGrey">
-                <color rgba="0.7 0.7 0.7 1.0" />
-            </material>
-            <origin rpy="0 0 0" xyz="0 0 0.127" />
-        </collision>
-        <collision>
-            <geometry>
-                <box size="1.55 1.55 1.1"/>
-            </geometry>
-            <material name="Green">
-                <color rgba="0.0 0.5 0.0 1.0" />
-            </material>
-            <origin rpy="0 0 0" xyz="0 1 0.55" />
-        </collision>
-        <inertial>
-            <mass value="0.1" />
-            <inertia ixx="0.03" iyy="0.03" izz="0.03" ixy="0.0" ixz="0.0" iyz="0.0" />
-        </inertial>
     <link name="${prefix}sander_center_link" />
-    <link name="${prefix}sander_intermediate_link">
-      <visual>
-          <geometry>
-              <cylinder length="0.025" radius="0.06425" />
-          </geometry>
-          <origin rpy="0 0 0" xyz="0 0 0" />
-      </visual>
-      <collision>
-          <geometry>
-              <cylinder length="0.025" radius="0.06425" />
-          </geometry>
-          <origin rpy="0 0 0" xyz="0 0 0" />
-      </collision>
-    </link>
-    <joint name="${prefix}sander_intermediate_to_sander_center_link" type="fixed">
-      <parent link="${prefix}sander_intermediate_link" />
-      <child link="${prefix}sander_center_link" />
-<!--        <origin xyz="0 0.16578 0.01902" rpy="-0.785 0 0" />-->
-<!--        <origin xyz="0 0.162 0.015" rpy="-0.785 0 0" />-->
-<!--        <origin xyz="0 0.04612 -0.03371" rpy="-2.355 0 0" />-->
-      <origin  xyz="0.0 0.0 0.0125" rpy="0.0 0.0 0.0"/>
-    </joint>
-    <joint name="${prefix}tool0_to_sander_intermediate_link" type="fixed">
+    <joint name="${prefix}tool0_to_sander_center_link" type="fixed">
         <parent link="${prefix}eoat_link" />
-        <child link="${prefix}sander_intermediate_link" />
+        <child link="${prefix}sander_center_link" />
 <!--        <origin xyz="0 0.16578 0.01902" rpy="-0.785 0 0" />-->
 <!--        <origin xyz="0 0.162 0.015" rpy="-0.785 0 0" />-->
@@ -496,5 +410,5 @@
         <child link="${prefix}camera_link"/>
     </joint>
-    <link name="${prefix}part" >
+<!--    <link name="${prefix}part" >
         <visual>
             <geometry>
@@ -506,5 +420,5 @@
             <origin rpy="0 0 0" xyz="0 0 -0.25" />
         </visual>
-<!--        <visual>
+        <visual>
             <origin rpy="0 0 0" xyz="0 0 0" />
             <geometry>
@@ -519,12 +433,12 @@
                 <mesh filename="package://crs_support/meshes/Parts/collision/part1_ch.stl" />
             </geometry>
-        </collision>-->
-    </link>
-    <joint name="${prefix}robot_stand_to_part_joint" type= "fixed">
-<!--        <origin xyz="-0.5 0.5 1.3" rpy= "1.571 -1.571 0"/>-->
-        <origin xyz="-0.25 0.5 1.15" rpy= "0.0 0.0 0"/>
-        <parent link="${prefix}robot_stand"/>
+        </collision>
+    </link>-->
+<!--    <joint name="${prefix}robot_stand_to_part_joint" type= "fixed">
+        <origin xyz="-0.5 0.5 1.3" rpy= "1.571 -1.571 0"/>
+        <origin xyz="0.25 -0.28 0.0" rpy= "0.0 0.0 1.571"/>
+        <parent link="table"/>
         <child link="${prefix}part"/>
-    </joint>
+    </joint>-->
     <transmission name="trans_shoulder_pan_joint">
         <type>transmission_interface/SimpleTransmission</type>

Commit message: code clean up, removed extra files

File: crs_support/urdf/swri_demo.urdf.xacro (robot description, xacro)
@@ -2,4 +2,87 @@
 <robot name="crs" xmlns:xacro="http://ros.org/wiki/xacro">
   <xacro:macro name="crs_workcell" params="prefix:=^|''">
+  <xacro:arg name="table_size" default="3.0"/>
+    <link name="world"/>
+    <link name="table">
+      <visual>
+        <origin xyz="0 0 -0.05"/>
+        <geometry>
+          <box size="$(arg table_size) $(arg table_size) 0.1"/>
+        </geometry>
+        <material name="StainlessSteel">
+          <color rgba="0.8 0.8 0.8 0.9"/>
+        </material>
+      </visual>
+      <collision>
+        <origin xyz="0 0 -0.05"/>
+        <geometry>
+          <box size="$(arg table_size) $(arg table_size) 0.1"/>
+        </geometry>
+      </collision>
+    </link>
+    <joint name="world_to_table_joint" type="fixed">
+<!--      <origin xyz="0 0 -0.363"/>-->
+      <origin xyz="0 0 -0.353"/>
+<!--      <origin xyz="0 0 -0.385"/>-->
+      <parent link="world"/>
+      <child link="table"/>
+    </joint>
+  <!--  <link name="${prefix}part"/>
+    <joint name="table_to_part" type="fixed">
+      <origin xyz="0.0 -0.875 -0.008" />
+      <parent link="table"/>
+      <child link="${prefix}part"/>
+    </joint>-->
+    <link name="robot_stand">
+      <visual>
+        <origin xyz="0 0 -0.1905"/>
+        <geometry>
+          <box size="0.35 0.35 0.381"/>
+        </geometry>
+      </visual>
+      <collision>
+        <origin xyz="0 0 -0.1905"/>
+        <geometry>
+          <box size="0.35 0.35 0.381"/>
+        </geometry>
+      </collision>
+    </link>
+    <joint name="table_to_robot_stand" type="fixed">
+      <origin xyz="0.0 0.0 0.0" rpy="0.0 0.0 3.1415"/>
+      <parent link="world"/>
+      <child link="robot_stand"/>
+    </joint>
+    <link name="${prefix}external_walls">
+      <visual>
+        <origin xyz="0 -1.2 -0.36"/>
+        <geometry>
+          <box size="$(arg table_size) 0.4 0.5"/>
+        </geometry>
+        <material name="StainlessSteel"/>
+      </visual>
+      <collision>
+        <origin xyz="0 -1.2 -0.36"/>
+        <geometry>
+          <box size="$(arg table_size) 0.4 0.5"/>
+        </geometry>
+      </collision>
+      <visual>
+        <origin xyz="0 0.765 0"/>
+        <geometry>
+          <box size="$(arg table_size) 0.1 $(arg table_size)"/>
+        </geometry>
+      </visual>
+      <collision>
+        <origin xyz="0 0.765 0"/>
+        <geometry>
+          <box size="$(arg table_size) 0.1 $(arg table_size)"/>
+        </geometry>
+      </collision>
+    </link>
+    <joint name="table_to_external_walls" type="fixed">
+      <origin xyz="0.0 0.0 0.0" rpy="0.0 0.0 0.0"/>
+      <parent link="world"/>
+      <child link="${prefix}external_walls"/>
+    </joint>
     <link name="${prefix}base_link">
         <visual>
@@ -222,4 +305,9 @@
     </link>
     <link name="${prefix}base" />
+    <joint name="table_to_ur" type="fixed">
+      <origin xyz="0.0 0.0 0.0" rpy="0.0 0.0 3.1415"/>
+      <parent link="world"/>
+      <child link="${prefix}base"/>
+    </joint>
     <joint name="${prefix}base_link-base_fixed_joint" type="fixed">
         <origin rpy="0 0 0" xyz="0 0 0" />
@@ -234,117 +322,71 @@
     </joint>
     <link name="${prefix}eoat_link">
-        <visual>
-            <geometry>
-                <mesh filename="package://crs_support/meshes/end_effector/visual/full_ee_v4.stl" />
-            </geometry>
-            <material name="Orange">
-                <color rgba="1.0 0.4 0.0 1.0" />
-            </material>
-        </visual>
-        <collision>
-            <geometry>
-                <mesh filename="package://crs_support/meshes/end_effector/collision/full_ee_v4_collision.stl" />
-            </geometry>
-        </collision>
-        <inertial>
-            <mass value="0.01" />
-            <origin rpy="0 0 0" xyz="0.0 0.0 0.0" />
-            <inertia ixx="0.000526462289415" ixy="0.0" ixz="0.0" iyy="0.000526462289415" iyz="0.0" izz="0.000568125" />
-        </inertial>
+      <visual>
+          <geometry>
+              <mesh filename="package://crs_support/meshes/end_effector/visual/full_ee_v4.stl" />
+          </geometry>
+          <material name="Orange">
+              <color rgba="1.0 0.4 0.0 1.0" />
+          </material>
+      </visual>
+      <collision>
+          <geometry>
+              <mesh filename="package://crs_support/meshes/end_effector/collision/full_ee_v4_collision.stl" />
+          </geometry>
+      </collision>
+<!--      <inertial>
+        <origin xyz="8.625E-08 -4.6583E-06 0.03145" rpy="0 0 0" />
+        <origin xyz="0 0 0" rpy="0 0 0" />
+        <mass value="0.22652" />
+        <inertia ixx="0.00020005" ixy="-4.2442E-10" ixz="-2.9069E-10" iyy="0.00017832" iyz="-3.4402E-08" izz="0.00013478" />
+      </inertial>
+      <visual>
+        <origin xyz="0 0 0" rpy="0 0 0" />
+        <geometry>
+          <mesh filename="package://crs_support/meshes/end_effector/visual/ee1.stl" />
+        </geometry>
+        <material name="">
+          <color rgba="0.1 0.1 0.1 1" />
+        </material>
+      </visual>
+      <visual>
+        <origin xyz="0 0 0" rpy="0 0 0" />
+        <geometry>
+          <mesh filename="package://crs_support/meshes/end_effector/visual/ee2.stl" />
+        </geometry>
+        <material name="">
+          <color rgba="0.1 0.1 0.1 1" />
+        </material>
+      </visual>
+      <visual>
+        <origin xyz="0 0 0" rpy="0 0 0" />
+        <geometry>
+          <mesh filename="package://crs_support/meshes/end_effector/visual/ee3.stl" />
+        </geometry>
+        <material name="">
+          <color rgba="0.1 0.1 0.1 1" />
+        </material>
+      </visual>
+      <collision>
+        <origin xyz="0 0 0" rpy="0 0 0" />
+        <geometry>
+          <mesh filename="package://crs_support/meshes/end_effector/visual/ee1.stl" />
+        </geometry>
+      </collision>-->
     </link>
     <joint name="${prefix}tool0_to_eoat_link" type="fixed">
         <parent link="${prefix}tool0" />
         <child link="${prefix}eoat_link" />
-        <origin rpy="0.0 0.0 0" xyz="0.00 0.00 0.00" />
-    </joint>
-    <link name="${prefix}robot_stand">
-        <visual>
-            <geometry>
-                <box size="0.4318 0.4318 1.1"/>
-            </geometry>
-            <material name="LightGrey">
-                <color rgba="0.7 0.7 0.7 1.0" />
-            </material>
-            <origin rpy="0 0 0" xyz="0 0 0.55" />
-        </visual>
-        <visual>
-            <geometry>
-                <box size="0.889 0.889 0.7112"/>
-            </geometry>
-            <material name="LightGrey">
-                <color rgba="0.7 0.7 0.7 1.0" />
-            </material>
-            <origin rpy="0 0 0" xyz="0 0 0.3556" />
-        </visual>
-        <visual>
-            <geometry>
-                <box size="1.55 1.55 0.254"/>
-            </geometry>
-            <material name="LightGrey">
-                <color rgba="0.7 0.7 0.7 1.0" />
-            </material>
-            <origin rpy="0 0 0" xyz="0 0 0.127" />
-        </visual>
-        <visual>
-            <geometry>
-                <box size="1.55 1.55 1.1"/>
-            </geometry>
-            <material name="Green">
-                <color rgba="0.0 0.5 0.0 1.0" />
-            </material>
-            <origin rpy="0 0 0" xyz="0 1 0.55" />
-        </visual>
-        <collision>
-            <geometry>
-                <box size="0.4318 0.4318 1.1"/>
-            </geometry>
-            <material name="LightGrey">
-                <color rgba="0.7 0.7 0.7 1.0" />
-            </material>
-            <origin rpy="0 0 0" xyz="0 0 0.55" />
-        </collision>
-        <collision>
-            <geometry>
-                <box size="0.889 0.889 0.7112"/>
-            </geometry>
-            <material name="LightGrey">
-                <color rgba="0.7 0.7 0.7 1.0" />
-            </material>
-            <origin rpy="0 0 0" xyz="0 0 0.3556" />
-        </collision>
-        <collision>
-            <geometry>
-                <box size="1.55 1.55 0.254"/>
-            </geometry>
-            <material name="LightGrey">
-                <color rgba="0.7 0.7 0.7 1.0" />
-            </material>
-            <origin rpy="0 0 0" xyz="0 0 0.127" />
-        </collision>
-        <collision>
-            <geometry>
-                <box size="1.55 1.55 1.1"/>
-            </geometry>
-            <material name="Green">
-                <color rgba="0.0 0.5 0.0 1.0" />
-            </material>
-            <origin rpy="0 0 0" xyz="0 1 0.55" />
-        </collision>
-        <inertial>
-            <mass value="0.1" />
-            <inertia ixx="0.03" iyy="0.03" izz="0.03" ixy="0.0" ixz="0.0" iyz="0.0" />
-        </inertial>
-    </link>
-    <joint name="${prefix}robot_base_joint" type="fixed">
-        <parent link="robot_stand" />
-        <child link="base" />
-        <origin rpy="0 0 0" xyz="0 0 1.0922" />
-        <limit effort="1.0" lower="-0.1" upper="1.9" velocity=".01" />
-    </joint>
-    <link name="world" />
-    <joint name="${prefix}robot_stand_joint" type="fixed">
-        <parent link="world" />
-        <child link="${prefix}robot_stand" />
-        <origin rpy="0 0 0" xyz="0 0 0" />
+<!--        <origin xyz="0 0 0" rpy="1.57 0 -1.57" />-->
+        <origin xyz="0 0 0" rpy="0 0 0" />
+    </joint>
+    <link name="${prefix}sander_center_link" />
+    <joint name="${prefix}tool0_to_sander_center_link" type="fixed">
+        <parent link="${prefix}eoat_link" />
+        <child link="${prefix}sander_center_link" />
+<!--        <origin xyz="0 0.16578 0.01902" rpy="-0.785 0 0" />-->
+<!--        <origin xyz="0 0.162 0.015" rpy="-0.785 0 0" />-->
+<!--        <origin xyz="0 0.04612 -0.03371" rpy="-2.355 0 0" />-->
+        <origin xyz="0.0 -0.15497 0.17503" rpy="0.7854 0.0 0.0"/>
     </joint>
     <link name="${prefix}gazebo_camera_link" />
@@ -361,11 +403,12 @@
         <child link="${prefix}camera_link_optical"/>
     </joint>
-    <link name="${prefix}sander_center_link" />
-    <joint name="${prefix}sander_joint" type = "fixed">
-        <origin xyz="0.0 -0.15497 0.17503" rpy="0.7854 0.0 0.0"/>
-        <parent link="${prefix}eoat_link"/>
-        <child link="${prefix}sander_center_link" />
-    </joint>
-    <link name="${prefix}part" >
+    <link name="${prefix}camera_link" />
+    <joint name="${prefix}camera_link_joint" type="fixed">
+<!--        <origin xyz="0.001 0.015 0.0" rpy="-1.57 1.57 0"/>-->
+        <origin xyz="0.0 0.0 0.0" rpy="1.57 -1.57 0"/>
+        <parent link="${prefix}camera_link_optical"/>
+        <child link="${prefix}camera_link"/>
+    </joint>
+<!--    <link name="${prefix}part" >
         <visual>
             <geometry>
@@ -377,5 +420,5 @@
             <origin rpy="0 0 0" xyz="0 0 -0.25" />
         </visual>
-<!--        <visual>
+        <visual>
             <origin rpy="0 0 0" xyz="0 0 0" />
             <geometry>
@@ -390,12 +433,12 @@
                 <mesh filename="package://crs_support/meshes/Parts/collision/part1_ch.stl" />
             </geometry>
-        </collision>-->
-    </link>
-    <joint name="${prefix}robot_stand_to_part_joint" type= "fixed">
-<!--        <origin xyz="-0.5 0.5 1.3" rpy= "1.571 -1.571 0"/>-->
-        <origin xyz="-0.25 0.5 1.15" rpy= "0.0 0.0 0"/>
-        <parent link="${prefix}robot_stand"/>
+        </collision>
+    </link>-->
+<!--    <joint name="${prefix}robot_stand_to_part_joint" type= "fixed">
+        <origin xyz="-0.5 0.5 1.3" rpy= "1.571 -1.571 0"/>
+        <origin xyz="0.25 -0.28 0.0" rpy= "0.0 0.0 1.571"/>
+        <parent link="table"/>
         <child link="${prefix}part"/>
-    </joint>
+    </joint>-->
     <transmission name="trans_shoulder_pan_joint">
         <type>transmission_interface/SimpleTransmission</type>

Commit message: Minor fixes for integration

File: crs_support/urdf/swri_demo.urdf.xacro (robot description, xacro)
@@ -54,17 +54,4 @@
     </joint>
     <link name="${prefix}external_walls">
-      <visual>
-        <origin xyz="0 -1.2 -0.36"/>
-        <geometry>
-          <box size="$(arg table_size) 0.4 0.5"/>
-        </geometry>
-        <material name="StainlessSteel"/>
-      </visual>
-      <collision>
-        <origin xyz="0 -1.2 -0.36"/>
-        <geometry>
-          <box size="$(arg table_size) 0.4 0.5"/>
-        </geometry>
-      </collision>
       <visual>
         <origin xyz="0 0.765 0"/>
@@ -382,7 +369,29 @@
     </joint>
     <link name="${prefix}sander_center_link" />
-    <joint name="${prefix}tool0_to_sander_center_link" type="fixed">
+    <link name="${prefix}sander_intermediate_link">
+      <visual>
+          <geometry>
+              <cylinder length="0.025" radius="0.06425" />
+          </geometry>
+          <origin rpy="0 0 0" xyz="0 0 0" />
+      </visual>
+      <collision>
+          <geometry>
+              <cylinder length="0.025" radius="0.06425" />
+          </geometry>
+          <origin rpy="0 0 0" xyz="0 0 0" />
+      </collision>
+    </link>
+    <joint name="${prefix}sander_intermediate_to_sander_center_link" type="fixed">
+      <parent link="${prefix}sander_intermediate_link" />
+      <child link="${prefix}sander_center_link" />
+<!--        <origin xyz="0 0.16578 0.01902" rpy="-0.785 0 0" />-->
+<!--        <origin xyz="0 0.162 0.015" rpy="-0.785 0 0" />-->
+<!--        <origin xyz="0 0.04612 -0.03371" rpy="-2.355 0 0" />-->
+      <origin  xyz="0.0 0.0 0.0125" rpy="0.0 0.0 0.0"/>
+    </joint>
+    <joint name="${prefix}tool0_to_sander_intermediate_link" type="fixed">
         <parent link="${prefix}eoat_link" />
-        <child link="${prefix}sander_center_link" />
+        <child link="${prefix}sander_intermediate_link" />
 <!--        <origin xyz="0 0.16578 0.01902" rpy="-0.785 0 0" />-->
 <!--        <origin xyz="0 0.162 0.015" rpy="-0.785 0 0" />-->
@@ -410,35 +419,4 @@
         <child link="${prefix}camera_link"/>
     </joint>
-<!--    <link name="${prefix}part" >
-        <visual>
-            <geometry>
-                <box size="0.25 0.25 0.5"/>
-            </geometry>
-            <material name="Green">
-                <color rgba="0.0 0.7 0.0 1.0" />
-            </material>
-            <origin rpy="0 0 0" xyz="0 0 -0.25" />
-        </visual>
-        <visual>
-            <origin rpy="0 0 0" xyz="0 0 0" />
-            <geometry>
-                <mesh filename="package://crs_support/meshes/Parts/visual/part1_ch.stl" />
-            </geometry>
-            <material name="Green">
-                <color rgba="0.0 0.7 0.0 1.0" />
-            </material>
-        </visual>
-        <collision>
-            <geometry>
-                <mesh filename="package://crs_support/meshes/Parts/collision/part1_ch.stl" />
-            </geometry>
-        </collision>
-    </link>-->
-<!--    <joint name="${prefix}robot_stand_to_part_joint" type= "fixed">
-        <origin xyz="-0.5 0.5 1.3" rpy= "1.571 -1.571 0"/>
-        <origin xyz="0.25 -0.28 0.0" rpy= "0.0 0.0 1.571"/>
-        <parent link="table"/>
-        <child link="${prefix}part"/>
-    </joint>-->
     <transmission name="trans_shoulder_pan_joint">
         <type>transmission_interface/SimpleTransmission</type>

Commit message: Minor fixes for integration

File: crs_support/urdf/swri_demo.urdf.xacro (robot description, xacro)
@@ -54,5 +54,5 @@
     </joint>
     <link name="${prefix}external_walls">
-      <visual>
+      <!--<visual>
         <origin xyz="0 -1.2 -0.36"/>
         <geometry>
@@ -66,5 +66,5 @@
           <box size="$(arg table_size) 0.4 0.5"/>
         </geometry>
-      </collision>
+      </collision>-->
       <visual>
         <origin xyz="0 0.765 0"/>
@@ -382,7 +382,29 @@
     </joint>
     <link name="${prefix}sander_center_link" />
-    <joint name="${prefix}tool0_to_sander_center_link" type="fixed">
+    <link name="${prefix}sander_intermediate_link">
+      <visual>
+          <geometry>
+              <cylinder length="0.025" radius="0.06425" />
+          </geometry>
+          <origin rpy="0 0 0" xyz="0 0 0" />
+      </visual>
+      <collision>
+          <geometry>
+              <cylinder length="0.025" radius="0.06425" />
+          </geometry>
+          <origin rpy="0 0 0" xyz="0 0 0" />
+      </collision>
+    </link>
+    <joint name="${prefix}sander_intermediate_to_sander_center_link" type="fixed">
+      <parent link="${prefix}sander_intermediate_link" />
+      <child link="${prefix}sander_center_link" />
+<!--        <origin xyz="0 0.16578 0.01902" rpy="-0.785 0 0" />-->
+<!--        <origin xyz="0 0.162 0.015" rpy="-0.785 0 0" />-->
+<!--        <origin xyz="0 0.04612 -0.03371" rpy="-2.355 0 0" />-->
+      <origin  xyz="0.0 0.0 0.0125" rpy="0.0 0.0 0.0"/>
+    </joint>
+    <joint name="${prefix}tool0_to_sander_intermediate_link" type="fixed">
         <parent link="${prefix}eoat_link" />
-        <child link="${prefix}sander_center_link" />
+        <child link="${prefix}sander_intermediate_link" />
 <!--        <origin xyz="0 0.16578 0.01902" rpy="-0.785 0 0" />-->
 <!--        <origin xyz="0 0.162 0.015" rpy="-0.785 0 0" />-->
