Commit message: removed excess commented out code

File: crs_support/urdf/swri_demo.urdf.xacro (robot description, xacro)
@@ -54,17 +54,4 @@
     </joint>
     <link name="${prefix}external_walls">
-      <!--<visual>
-        <origin xyz="0 -1.2 -0.36"/>
-        <geometry>
-          <box size="$(arg table_size) 0.4 0.5"/>
-        </geometry>
-        <material name="StainlessSteel"/>
-      </visual>
-      <collision>
-        <origin xyz="0 -1.2 -0.36"/>
-        <geometry>
-          <box size="$(arg table_size) 0.4 0.5"/>
-        </geometry>
-      </collision>-->
       <visual>
         <origin xyz="0 0.765 0"/>
@@ -432,35 +419,4 @@
         <child link="${prefix}camera_link"/>
     </joint>
-<!--    <link name="${prefix}part" >
-        <visual>
-            <geometry>
-                <box size="0.25 0.25 0.5"/>
-            </geometry>
-            <material name="Green">
-                <color rgba="0.0 0.7 0.0 1.0" />
-            </material>
-            <origin rpy="0 0 0" xyz="0 0 -0.25" />
-        </visual>
-        <visual>
-            <origin rpy="0 0 0" xyz="0 0 0" />
-            <geometry>
-                <mesh filename="package://crs_support/meshes/Parts/visual/part1_ch.stl" />
-            </geometry>
-            <material name="Green">
-                <color rgba="0.0 0.7 0.0 1.0" />
-            </material>
-        </visual>
-        <collision>
-            <geometry>
-                <mesh filename="package://crs_support/meshes/Parts/collision/part1_ch.stl" />
-            </geometry>
-        </collision>
-    </link>-->
-<!--    <joint name="${prefix}robot_stand_to_part_joint" type= "fixed">
-        <origin xyz="-0.5 0.5 1.3" rpy= "1.571 -1.571 0"/>
-        <origin xyz="0.25 -0.28 0.0" rpy= "0.0 0.0 1.571"/>
-        <parent link="table"/>
-        <child link="${prefix}part"/>
-    </joint>-->
     <transmission name="trans_shoulder_pan_joint">
         <type>transmission_interface/SimpleTransmission</type>

Commit message: changed camera frame locations

File: crs_support/urdf/swri_demo.urdf.xacro (robot description, xacro)
@@ -407,5 +407,5 @@
     <link name="${prefix}camera_link_optical" />
     <joint name="${prefix}camera_optical_joint" type="fixed">
-        <origin xyz="-0.00345 0.070793 0.077409" rpy="-0.7854 0 0"/>
+        <origin xyz="-0.022 0.079773 0.065" rpy="-0.7854 0 0"/>
         <parent link="${prefix}eoat_link"/>
         <!-- <parent link="${prefix}gazebo_camera_link"/> -->

Commit message: updated camera position

File: crs_support/urdf/swri_demo.urdf.xacro (robot description, xacro)
@@ -14,10 +14,10 @@
         </material>
       </visual>
-<!--      <collision>
+      <collision>
         <origin xyz="0 0 -0.05"/>
         <geometry>
           <box size="$(arg table_size) $(arg table_size) 0.1"/>
         </geometry>
-      </collision>-->
+      </collision>
     </link>
     <joint name="world_to_table_joint" type="fixed">
@@ -407,5 +407,5 @@
     <link name="${prefix}camera_link_optical" />
     <joint name="${prefix}camera_optical_joint" type="fixed">
-        <origin xyz="-0.022 0.079773 0.065" rpy="-0.7854 0 0"/>
+        <origin xyz="-0.021 0.0797 0.06525" rpy="-0.7854 0 0"/>
         <parent link="${prefix}eoat_link"/>
         <!-- <parent link="${prefix}gazebo_camera_link"/> -->
@@ -415,5 +415,5 @@
     <joint name="${prefix}camera_link_joint" type="fixed">
 <!--        <origin xyz="0.001 0.015 0.0" rpy="-1.57 1.57 0"/>-->
-        <origin xyz="0.0 0.0 0.0" rpy="1.57 -1.57 0"/>
+        <origin xyz="0.00 0.0 0.003" rpy="1.57 -1.57 0.0"/>
         <parent link="${prefix}camera_link_optical"/>
         <child link="${prefix}camera_link"/>

Commit message: saved realsense workcell configuration

File: crs_support/urdf/swri_demo.urdf.xacro (robot description, xacro)
@@ -22,7 +22,5 @@
     </link>
     <joint name="world_to_table_joint" type="fixed">
-<!--      <origin xyz="0 0 -0.363"/>-->
-      <origin xyz="0 0 -0.353"/>
-<!--      <origin xyz="0 0 -0.385"/>-->
+      <origin xyz="0 0 ${-0.353 - 0.010}"/>
       <parent link="world"/>
       <child link="table"/>
@@ -391,5 +389,6 @@
     <link name="${prefix}camera_link_optical" />
     <joint name="${prefix}camera_optical_joint" type="fixed">
-        <origin xyz="-0.021 0.0797 0.06525" rpy="-0.7854 0 0"/>
+    	<!-- <origin xyz="-0.021 0.0797 0.06525" rpy="-0.7854 0 0"/> --> <!-- framos config -->
+        <origin xyz="-0.021 0.0797 0.05" rpy="-0.7854 0 0"/><!-- realsense config -->
         <parent link="${prefix}eoat_link"/>
         <child link="${prefix}camera_link_optical"/>
