Commit message: uses xacro to allow namespacing of links and joints for preview purposes, creates soft link into .gazebo/models directory

File: crs_support/urdf/crs.urdf.xacro (robot description, xacro)
@@ -1,5 +1,6 @@
 <?xml version="1.0" encoding="utf-8" ?>
 <robot name="crs" xmlns:xacro="http://ros.org/wiki/xacro">
-    <link name="base_link">
+  <xacro:macro name="crs_workcell" params="prefix:=^|''">
+    <link name="${prefix}base_link">
         <visual>
             <origin rpy="0 0 3.14159265359" xyz="0 0 0" />
@@ -23,7 +24,7 @@
         </inertial>
     </link>
-    <joint name="shoulder_pan_joint" type="revolute">
-        <parent link="base_link" />
-        <child link="shoulder_link" />
+    <joint name="${prefix}shoulder_pan_joint" type="revolute">
+        <parent link="${prefix}base_link" />
+        <child link="${prefix}shoulder_link" />
         <origin rpy="0 0 3.14159249728" xyz="0 0 0.180920744391" />
         <axis xyz="0 0 1" />
@@ -31,5 +32,5 @@
         <dynamics damping="0.0" friction="0.0" />
     </joint>
-    <link name="shoulder_link">
+    <link name="${prefix}shoulder_link">
         <visual>
             <origin rpy="0 0 3.14159265359" xyz="0 0 0" />
@@ -53,7 +54,7 @@
         </inertial>
     </link>
-    <joint name="shoulder_lift_joint" type="revolute">
-        <parent link="shoulder_link" />
-        <child link="upper_arm_link" />
+    <joint name="${prefix}shoulder_lift_joint" type="revolute">
+        <parent link="${prefix}shoulder_link" />
+        <child link="${prefix}upper_arm_link" />
         <origin rpy="1.57065145242 0 -2.70337965131e-06" xyz="0.00013292041689 0 0" />
         <axis xyz="0 0 1" />
@@ -61,5 +62,5 @@
         <dynamics damping="0.0" friction="0.0" />
     </joint>
-    <link name="upper_arm_link">
+    <link name="${prefix}upper_arm_link">
         <visual>
             <origin rpy="1.57079632679 0 -1.57079632679" xyz="0 0 0.1762" />
@@ -83,7 +84,7 @@
         </inertial>
     </link>
-    <joint name="elbow_joint" type="revolute">
-        <parent link="upper_arm_link" />
-        <child link="forearm_link" />
+    <joint name="${prefix}elbow_joint" type="revolute">
+        <parent link="${prefix}upper_arm_link" />
+        <child link="${prefix}forearm_link" />
         <origin rpy="3.14047492209 3.14117521433 3.14159104748" xyz="-0.611971344601 0 0" />
         <axis xyz="0 0 1" />
@@ -91,5 +92,5 @@
         <dynamics damping="0.0" friction="0.0" />
     </joint>
-    <link name="forearm_link">
+    <link name="${prefix}forearm_link">
         <visual>
             <origin rpy="1.57079632679 0 -1.57079632679" xyz="0 0 0.0393" />
@@ -113,7 +114,7 @@
         </inertial>
     </link>
-    <joint name="wrist_1_joint" type="revolute">
-        <parent link="forearm_link" />
-        <child link="wrist_1_link" />
+    <joint name="${prefix}wrist_1_joint" type="revolute">
+        <parent link="${prefix}forearm_link" />
+        <child link="${prefix}wrist_1_link" />
         <origin rpy="3.13872123266 -3.14053617519 3.14158723656" xyz="-0.571064941288 0.000500820247035 0.174414995927" />
         <axis xyz="0 0 1" />
@@ -121,5 +122,5 @@
         <dynamics damping="0.0" friction="0.0" />
     </joint>
-    <link name="wrist_1_link">
+    <link name="${prefix}wrist_1_link">
         <visual>
             <origin rpy="1.57079632679 0 0" xyz="0 0 -0.135" />
@@ -143,7 +144,7 @@
         </inertial>
     </link>
-    <joint name="wrist_2_joint" type="revolute">
-        <parent link="wrist_1_link" />
-        <child link="wrist_2_link" />
+    <joint name="${prefix}wrist_2_joint" type="revolute">
+        <parent link="${prefix}wrist_1_link" />
+        <child link="${prefix}wrist_2_link" />
         <origin rpy="1.57117550062 0 -9.13444434245e-07" xyz="5.96404309737e-05 -0.119843553735 -4.54415414531e-05" />
         <axis xyz="0 0 1" />
@@ -151,5 +152,5 @@
         <dynamics damping="0.0" friction="0.0" />
     </joint>
-    <link name="wrist_2_link">
+    <link name="${prefix}wrist_2_link">
         <visual>
             <origin rpy="0 0 0" xyz="0 0 -0.12" />
@@ -173,7 +174,7 @@
         </inertial>
     </link>
-    <joint name="wrist_3_joint" type="revolute">
-        <parent link="wrist_2_link" />
-        <child link="wrist_3_link" />
+    <joint name="${prefix}wrist_3_joint" type="revolute">
+        <parent link="${prefix}wrist_2_link" />
+        <child link="${prefix}wrist_3_link" />
         <origin rpy="1.57170379674 3.14159265359 3.14159254819" xyz="1.57784168351e-05 0.115533666641 0.000104843358957" />
         <axis xyz="0 0 1" />
@@ -181,5 +182,5 @@
         <dynamics damping="0.0" friction="0.0" />
     </joint>
-    <link name="wrist_3_link">
+    <link name="${prefix}wrist_3_link">
         <visual>
             <origin rpy="1.57079632679 0 0" xyz="0 0 -0.1168" />
@@ -203,10 +204,10 @@
         </inertial>
     </link>
-    <joint name="ee_fixed_joint" type="fixed">
-        <parent link="wrist_3_link" />
-        <child link="ee_link" />
+    <joint name="${prefix}ee_fixed_joint" type="fixed">
+        <parent link="${prefix}wrist_3_link" />
+        <child link="${prefix}ee_link" />
         <origin rpy="0.0 -1.57079632679 1.57079632679" xyz="0.0 0.0 0.0" />
     </joint>
-    <link name="ee_link">
+    <link name="${prefix}ee_link">
         <collision>
             <geometry>
@@ -220,17 +221,17 @@
         </inertial>
     </link>
-    <link name="base" />
-    <joint name="base_link-base_fixed_joint" type="fixed">
+    <link name="${prefix}base" />
+    <joint name="${prefix}base_link-base_fixed_joint" type="fixed">
         <origin rpy="-1.571 0 0" xyz="0 0 0" />
-        <parent link="base" />
-        <child link="base_link" />
-    </joint>
-    <link name="tool0" />
-    <joint name="wrist_3_link-tool0_fixed_joint" type="fixed">
+        <parent link="${prefix}base" />
+        <child link="${prefix}base_link" />
+    </joint>
+    <link name="${prefix}tool0" />
+    <joint name="${prefix}wrist_3_link-tool0_fixed_joint" type="fixed">
         <origin rpy="0 0 0" xyz="0 0 0" />
-        <parent link="wrist_3_link" />
-        <child link="tool0" />
-    </joint>
-    <link name="eoat_link">
+        <parent link="${prefix}wrist_3_link" />
+        <child link="${prefix}tool0" />
+    </joint>
+    <link name="${prefix}eoat_link">
         <visual>
             <geometry>
@@ -252,10 +253,10 @@
         </inertial>
     </link>
-    <joint name="tool0_to_eoat_link" type="fixed">
-        <parent link="tool0" />
-        <child link="eoat_link" />
+    <joint name="${prefix}tool0_to_eoat_link" type="fixed">
+        <parent link="${prefix}tool0" />
+        <child link="${prefix}eoat_link" />
         <origin rpy="0.0 0.0 0" xyz="0.00 0.00 0.00" />
     </joint>
-    <link name="robot_stand">
+    <link name="${prefix}robot_stand">
         <visual>
             <origin rpy="1.57079632679 0 0" xyz="0 0 -0.1168" />
@@ -311,7 +312,7 @@
         </inertial>
     </link>
-    <joint name="robot_base_joint" type="fixed">
-        <parent link="robot_stand" />
-        <child link="base" />
+    <joint name="${prefix}robot_base_joint" type="fixed">
+        <parent link="${prefix}robot_stand" />
+        <child link="${prefix}base" />
         <origin rpy="0 1.571 0" xyz="0.036983 -2.0948 0.58 " />
         <axis xyz="1 0 0"/>
@@ -319,29 +320,29 @@
     </joint>
     <link name="world" />
-    <joint name="robot_stand_joint" type="fixed">
+    <joint name="${prefix}robot_stand_joint" type="fixed">
         <parent link="world" />
-        <child link="robot_stand" />
+        <child link="${prefix}robot_stand" />
         <origin rpy="-1.571 0 0" xyz="0 0 0" />
     </joint>
-    <link name="gazebo_camera_link" />
-    <joint name="gazebo_camera_joint" type="fixed">
+    <link name="${prefix}gazebo_camera_link" />
+    <joint name="${prefix}gazebo_camera_joint" type="fixed">
         <origin xyz="0.0 0.0 0.0" rpy="1.57 -1.57 0.0"/>
-        <parent link="camera_link_optical"/>
-        <child link="gazebo_camera_link"/>
-    </joint>
-    <link name="camera_link_optical" />
-    <joint name="camera_optical_joint" type="fixed">
+        <parent link="${prefix}camera_link_optical"/>
+        <child link="${prefix}gazebo_camera_link"/>
+    </joint>
+    <link name="${prefix}camera_link_optical" />
+    <joint name="${prefix}camera_optical_joint" type="fixed">
         <origin xyz="-0.00345 0.070793 0.077409" rpy="-0.7854 0 0"/>
-        <parent link="eoat_link"/>
-        <parent link="gazebo_camera_link"/>
-        <child link="camera_link_optical"/>
-    </joint>
-    <link name="sander_center_link" />
-    <joint name="sander_joint" type = "fixed">
+        <parent link="${prefix}eoat_link"/>
+        <!-- <parent link="${prefix}gazebo_camera_link"/> -->
+        <child link="${prefix}camera_link_optical"/>
+    </joint>
+    <link name="${prefix}sander_center_link" />
+    <joint name="${prefix}sander_joint" type = "fixed">
         <origin xyz="0.0 -0.1167 0.12664" rpy="0.7854 0.0 0.0"/>
-        <parent link="eoat_link"/>
-        <child link="sander_center_link" />
-    </joint>
-    <link name="part" >
+        <parent link="${prefix}eoat_link"/>
+        <child link="${prefix}sander_center_link" />
+    </joint>
+    <link name="${prefix}part" >
         <visual>
             <origin rpy="0 0 0" xyz="0 0 0" />
@@ -359,13 +360,13 @@
         </collision>-->
     </link>
-    <joint name="robot_stand_to_part_joint" type= "fixed">
+    <joint name="${prefix}robot_stand_to_part_joint" type= "fixed">
         <origin xyz="-0.439 -1.1 -0.14" rpy= "-3.1416 0.0 -1.571"/>
 <!--        <origin xyz="-0.439 -1.2 -0.14" rpy= "-3.1416 0.0 -1.571"/>-->
-        <parent link="robot_stand"/>
-        <child link="part"/>
+        <parent link="${prefix}robot_stand"/>
+        <child link="${prefix}part"/>
     </joint>
     <transmission name="trans_shoulder_pan_joint">
         <type>transmission_interface/SimpleTransmission</type>
-        <joint name="shoulder_pan_joint">
+        <joint name="${prefix}shoulder_pan_joint">
             <hardwareInterface>hardware_interface/EffortJointInterface</hardwareInterface>
         </joint>
@@ -377,5 +378,5 @@
     <transmission name="trans_shoulder_lift_joint">
         <type>transmission_interface/SimpleTransmission</type>
-        <joint name="shoulder_lift_joint">
+        <joint name="${prefix}shoulder_lift_joint">
             <hardwareInterface>hardware_interface/EffortJointInterface</hardwareInterface>
         </joint>
@@ -387,5 +388,5 @@
     <transmission name="trans_elbow_joint">
         <type>transmission_interface/SimpleTransmission</type>
-        <joint name="elbow_joint">
+        <joint name="${prefix}elbow_joint">
             <hardwareInterface>hardware_interface/EffortJointInterface</hardwareInterface>
         </joint>
@@ -397,5 +398,5 @@
     <transmission name="trans_wrist_1_joint">
         <type>transmission_interface/SimpleTransmission</type>
-        <joint name="wrist_1_joint">
+        <joint name="${prefix}wrist_1_joint">
             <hardwareInterface>hardware_interface/EffortJointInterface</hardwareInterface>
         </joint>
@@ -407,5 +408,5 @@
     <transmission name="trans_wrist_2_joint">
         <type>transmission_interface/SimpleTransmission</type>
-        <joint name="wrist_2_joint">
+        <joint name="${prefix}wrist_2_joint">
             <hardwareInterface>hardware_interface/EffortJointInterface</hardwareInterface>
         </joint>
@@ -417,5 +418,5 @@
     <transmission name="trans_wrist_3_joint">
         <type>transmission_interface/SimpleTransmission</type>
-        <joint name="wrist_3_joint">
+        <joint name="${prefix}wrist_3_joint">
             <hardwareInterface>hardware_interface/EffortJointInterface</hardwareInterface>
         </joint>
@@ -427,5 +428,5 @@
     <transmission name="trans_robot_base_joint">
         <type>transmission_interface/SimpleTransmission</type>
-        <joint name="robot_base_joint">
+        <joint name="${prefix}robot_base_joint">
             <hardwareInterface>hardware_interface/EffortJointInterface</hardwareInterface>
         </joint>
@@ -435,38 +436,38 @@
         </actuator>
     </transmission>
-    <gazebo reference="robot_stand">
-        <selfCollide>true</selfCollide>
-    </gazebo>
-    <gazebo reference="base_link">
-        <selfCollide>true</selfCollide>
-    </gazebo>
-    <gazebo reference="shoulder_link">
-        <selfCollide>true</selfCollide>
-    </gazebo>
-    <gazebo reference="upper_arm_link">
-        <selfCollide>true</selfCollide>
-    </gazebo>
-    <gazebo reference="wrist_1_joint">
-        <selfCollide>true</selfCollide>
-    </gazebo>
-    <gazebo reference="forearm_link">
-        <selfCollide>true</selfCollide>
-    </gazebo>
-    <gazebo reference="wrist_2_joint">
-        <selfCollide>true</selfCollide>
-    </gazebo>
-    <gazebo reference="wrist_3_joint">
-        <selfCollide>true</selfCollide>
-    </gazebo>
-    <gazebo reference="ee_link">
-        <selfCollide>true</selfCollide>
-    </gazebo>
-    <gazebo reference="eoat_link">
-        <selfCollide>true</selfCollide>
-    </gazebo>
-    <gazebo reference="tool0">
-        <selfCollide>true</selfCollide>
-    </gazebo>
-    <gazebo reference="gazebo_camera_link">
+    <gazebo reference="${prefix}robot_stand">
+        <selfCollide>true</selfCollide>
+    </gazebo>
+    <gazebo reference="${prefix}base_link">
+        <selfCollide>true</selfCollide>
+    </gazebo>
+    <gazebo reference="${prefix}shoulder_link">
+        <selfCollide>true</selfCollide>
+    </gazebo>
+    <gazebo reference="${prefix}upper_arm_link">
+        <selfCollide>true</selfCollide>
+    </gazebo>
+    <gazebo reference="${prefix}wrist_1_joint">
+        <selfCollide>true</selfCollide>
+    </gazebo>
+    <gazebo reference="${prefix}forearm_link">
+        <selfCollide>true</selfCollide>
+    </gazebo>
+    <gazebo reference="${prefix}wrist_2_joint">
+        <selfCollide>true</selfCollide>
+    </gazebo>
+    <gazebo reference="${prefix}wrist_3_joint">
+        <selfCollide>true</selfCollide>
+    </gazebo>
+    <gazebo reference="${prefix}ee_link">
+        <selfCollide>true</selfCollide>
+    </gazebo>
+    <gazebo reference="${prefix}eoat_link">
+        <selfCollide>true</selfCollide>
+    </gazebo>
+    <gazebo reference="${prefix}tool0">
+        <selfCollide>true</selfCollide>
+    </gazebo>
+    <gazebo reference="${prefix}gazebo_camera_link">
         <sensor type="depth" name="sensor_name">
           <!-- Set always_on only sensor, not on plugin -->
@@ -521,10 +522,10 @@
           </ros>
           <update_rate>50</update_rate>
-          <joint_name>shoulder_pan_joint</joint_name>
-          <joint_name>shoulder_lift_joint</joint_name>
-          <joint_name>elbow_joint</joint_name>
-          <joint_name>wrist_1_joint</joint_name>
-          <joint_name>wrist_2_joint</joint_name>
-          <joint_name>wrist_3_joint</joint_name>
+          <joint_name>${prefix}shoulder_pan_joint</joint_name>
+          <joint_name>${prefix}shoulder_lift_joint</joint_name>
+          <joint_name>${prefix}elbow_joint</joint_name>
+          <joint_name>${prefix}wrist_1_joint</joint_name>
+          <joint_name>${prefix}wrist_2_joint</joint_name>
+          <joint_name>${prefix}wrist_3_joint</joint_name>
         </plugin>
         <plugin name='gazebo_ros_joint_pose_trajectory' filename='libgazebo_ros_joint_pose_trajectory.so'>
@@ -536,3 +537,6 @@
         </plugin>
     </gazebo>
+  </xacro:macro>
+  <xacro:arg name="prefix" default=""/>
+  <xacro:crs_workcell prefix="$(arg prefix)"/>
 </robot>

Commit message: Added additional invisible barriers to urdf environment

File: crs_support/urdf/crs.urdf.xacro (robot description, xacro)
@@ -294,4 +294,16 @@
             </geometry>
             <origin rpy="0 0 0" xyz="-0.42 -1.1 -1.46" />
+        </collision>
+        <collision> Front Wall
+            <geometry>
+                <box size="0.1 2.14 2.65" />
+            </geometry>
+            <origin rpy="0 0 0" xyz="0.4 -1.1 -0.175" />
+        </collision>
+        <collision> Back Wall
+            <geometry>
+                <box size="0.1 2.14 2.65" />
+            </geometry>
+            <origin rpy="0 0 0" xyz="-1.25 -1.1 -0.175" />
         </collision>
         <collision> <!-- Top front beam-->

Commit message: Commented out part to be sanded from urdf

File: crs_support/urdf/crs.urdf.xacro (robot description, xacro)
@@ -356,5 +356,5 @@
         <child link="${prefix}sander_center_link" />
     </joint>
-    <link name="${prefix}part" >
+<!--    <link name="${prefix}part" >
         <visual>
             <origin rpy="0 0 0" xyz="0 0 0" />
@@ -366,16 +366,15 @@
             </material>
         </visual>
-<!--        <collision>
+        <collision>
             <geometry>
                 <mesh filename="package://crs_support/meshes/Parts/collision/part1_ch.stl" />
             </geometry>
-        </collision>-->
+        </collision>
     </link>
     <joint name="${prefix}robot_stand_to_part_joint" type= "fixed">
         <origin xyz="-0.439 -1.1 -0.14" rpy= "-3.1416 0.0 -1.571"/>
-<!--        <origin xyz="-0.439 -1.2 -0.14" rpy= "-3.1416 0.0 -1.571"/>-->
         <parent link="${prefix}robot_stand"/>
         <child link="${prefix}part"/>
-    </joint>
+    </joint>-->
     <transmission name="trans_shoulder_pan_joint">
         <type>transmission_interface/SimpleTransmission</type>

Commit message: Added new mockup and cart to urdf

File: crs_support/urdf/crs.urdf.xacro (robot description, xacro)
@@ -317,7 +317,7 @@
         <collision> Back Wall top beam
             <geometry>
-                <box size="0.1 0.15 3.0" />
-            </geometry>
-            <origin rpy="0 0 0" xyz="-2.06 -2.135 0.0" />
+                <box size="1.25 0.12 3.0" />
+            </geometry>
+            <origin rpy="0 0 0" xyz="0.38 -2.135 0.0" />
         </collision>
         <collision> Back Wall Half right
@@ -587,5 +587,5 @@
             <ros>
               <namespace>custom_ns</namespace>
-              <argument>camera/image_raw:=camera/image</argument>
+              <argument>camera/image_raw:=camera/custom_image</argument>
               <argument>camera/image_depth:=camera/custom_image_depth</argument>
               <argument>camera/camera_info:=camera/custom_info_raw</argument>

Commit message: Added ability to launch with simulation arg

File: crs_support/urdf/crs.urdf.xacro (robot description, xacro)
@@ -223,5 +223,6 @@
     <link name="${prefix}base" />
     <joint name="${prefix}base_link-base_fixed_joint" type="fixed">
-        <origin rpy="-1.571 0 0" xyz="0 0 0" />
+        <!--<origin rpy="-1.571 0 0" xyz="0 0 0" />-->
+        <origin rpy="0 0 0" xyz="0 0 0" />-->
         <parent link="${prefix}base" />
         <child link="${prefix}base_link" />
@@ -307,15 +308,27 @@
             <origin rpy="0 0 0" xyz="-2.06 -1.1 0.0" />
         </collision>
-        <collision> <!-- Top front beam-->
+<!--        <collision> < Top front beam>
             <geometry>
                 <box size="1.25 0.12 3.0" />
             </geometry>
             <origin rpy="0 0 0" xyz="0.38 -2.135 0.0" />
-        </collision>
+        </collision>-->
         <collision> <!-- Top back beam-->
             <geometry>
-                <box size="1.25 0.12 3.0" />
-            </geometry>
-            <origin rpy="0 0 0" xyz="-1.56 -2.135 0.0" />
+                <box size="0.4 0.12 3.0" />
+            </geometry>
+            <origin rpy="0 0 0" xyz="-0.98 -2.135 0.0" />
+        </collision>
+        <collision> <!-- Corner Bracket 1-->
+            <geometry>
+                <box size="1.25 0.12 1.25" />
+            </geometry>
+            <origin rpy="0 0.785 0" xyz="-2.06 -2.135 -1.33" />
+        </collision>
+        <collision> <!-- Corner Bracket 2-->
+            <geometry>
+                <box size="1.25 0.12 1.25" />
+            </geometry>
+            <origin rpy="0 0.785 0" xyz="-2.06 -2.135 1.38" />
         </collision>
         <inertial>
@@ -327,5 +340,6 @@
         <parent link="${prefix}robot_stand" />
         <child link="${prefix}base" />
-        <origin rpy="0 1.570796 0" xyz="-0.148896 -2.047406 0.6277 " />
+<!--        <origin rpy="-1.570796 1.570796 0" xyz="-0.148896 -2.047406 0.6277 " />-->
+        <origin rpy="-1.570796 1.570796 0" xyz="-1.050659 -2.047406 0.6277 " />
         <axis xyz="1 0 0"/>
         <limit effort="1.0" lower="-0.1" upper="1.9" velocity=".01" />
@@ -349,4 +363,11 @@
         <!-- <parent link="${prefix}gazebo_camera_link"/> -->
         <child link="${prefix}camera_link_optical"/>
+    </joint>
+    <link name="${prefix}camera_link" />
+    <joint name="${prefix}camera_link_joint" type="fixed">
+<!--        <origin xyz="0.001 0.015 0.0" rpy="-1.57 1.57 0"/>-->
+        <origin xyz="0.0 0.0 0.0" rpy="1.57 -1.57 0"/>
+        <parent link="${prefix}camera_link_optical"/>
+        <child link="${prefix}camera_link"/>
     </joint>
     <link name="${prefix}sander_center_link" />
@@ -510,12 +531,12 @@
             <ros>
               <namespace>custom_ns</namespace>
-              <argument>custom_camera/image_raw:=custom_camera/custom_image</argument>
-              <argument>custom_camera/image_depth:=custom_camera/custom_image_depth</argument>
-              <argument>custom_camera/camera_info:=custom_camera/custom_info_raw</argument>
-              <argument>custom_camera/camera_info_depth:=custom_camera/custom_info_depth</argument>
-              <argument>custom_camera/points:=custom_camera/custom_points</argument>
+              <argument>camera/image_raw:=camera/custom_image</argument>
+              <argument>camera/image_depth:=camera/custom_image_depth</argument>
+              <argument>camera/camera_info:=camera/custom_info_raw</argument>
+              <argument>camera/camera_info_depth:=camera/custom_info_depth</argument>
+              <argument>camera/points:=camera/pointcloud</argument>
             </ros>
             <!-- Set camera name. If empty, defaults to sensor name (i.e. "sensor_name") -->
-            <camera_name>custom_camera</camera_name>
+            <camera_name>camera</camera_name>
             <frame_name>camera_link_optical</frame_name>
             <!-- Set TF frame name. If empty, defaults to link name (i.e. "link_name") -->
