Commit message: modified robot base pose and collision geometry to better reflect actual system

File: crs_support/urdf/crs.urdf.xacro (robot description, xacro)
@@ -316,5 +316,5 @@
         <collision> <!-- Top back beam-->
             <geometry>
-                <box size="0.4 0.12 3.0" />
+                <box size="0.4 0.15 3.0" />
             </geometry>
             <origin rpy="0 0 0" xyz="-0.98 -2.135 0.0" />
@@ -340,6 +340,6 @@
         <parent link="${prefix}robot_stand" />
         <child link="${prefix}base" />
-<!--        <origin rpy="-1.570796 1.570796 0" xyz="-0.148896 -2.047406 0.6277 " />-->
-        <origin rpy="-1.570796 1.570796 0" xyz="-1.050659 -2.047406 0.6277 " />
+        <origin rpy="-1.570796 1.570796 0" xyz="-0.148896 -2.047406 0.6277 " />
+<!--        <origin rpy="-1.570796 1.570796 0" xyz="-1.030659 -2.037406 0.7977 " />-->
         <axis xyz="1 0 0"/>
         <limit effort="1.0" lower="-0.1" upper="1.9" velocity=".01" />

Commit message: Added end effector collision geometry and updated mockup collision geometry

File: crs_support/urdf/crs.urdf.xacro (robot description, xacro)
@@ -29,5 +29,6 @@
         <origin rpy="0 0 3.14159249728" xyz="0 0 0.180920744391" />
         <axis xyz="0 0 1" />
-        <limit effort="330.0" lower="-6.28318530718" upper="6.28318530718" velocity="3.14" />
+<!--        <limit effort="330.0" lower="-6.28318530718" upper="6.28318530718" velocity="3.14" />-->
+        <limit effort="330.0" lower="-4" upper="2.28" velocity="3.14" />
         <dynamics damping="0.0" friction="0.0" />
     </joint>
@@ -270,5 +271,5 @@
         </visual>
         <visual>
-            <origin rpy="1.57079632679 0 0" xyz="0 0 -0.1168" />
+            <origin rpy="1.57079632679 0 0" xyz="0.20 0 -0.1168" />
             <geometry>
                 <mesh filename="package://crs_support/meshes/Mockup/visual/mockup_cart_v4.stl" />
@@ -279,5 +280,5 @@
         </visual>
         <collision>
-            <origin rpy="1.57079632679 0 0" xyz="0 0 -0.1168" />
+            <origin rpy="1.57079632679 0 0" xyz="0.20 0 -0.1168" />
             <geometry>
                 <mesh filename="package://crs_support/meshes/Mockup/collision/Mockup3_6_Cart_collision.stl" />
@@ -302,9 +303,33 @@
             <origin rpy="0 0 0" xyz="0.85 -1.1 0.0" />
         </collision>
-        <collision> Back Wall
+        <!--<collision> Back Wall Full
             <geometry>
                 <box size="0.1 2.14 3.0" />
             </geometry>
             <origin rpy="0 0 0" xyz="-2.06 -1.1 0.0" />
+        </collision>-->
+        <collision> Back Wall bottom Half
+            <geometry>
+                <box size="0.1 1.1 3.0" />
+            </geometry>
+            <origin rpy="0 0 0" xyz="-2.06 -0.6 0.0" />
+        </collision>
+        <collision> Back Wall top beam
+            <geometry>
+                <box size="0.1 0.15 3.0" />
+            </geometry>
+            <origin rpy="0 0 0" xyz="-2.06 -2.135 0.0" />
+        </collision>
+        <collision> Back Wall Half right
+            <geometry>
+                <box size="0.1 0.3 0.7" />
+            </geometry>
+            <origin rpy="-0.786 0 0" xyz="-2.06 -1.9 1.15" />
+        </collision>
+        <collision> Back Wall Half left
+            <geometry>
+                <box size="0.1 0.3 0.7" />
+            </geometry>
+            <origin rpy="0.786 0 0" xyz="-2.06 -1.9 -1.15" />
         </collision>
 <!--        <collision> < Top front beam>
@@ -316,7 +341,7 @@
         <collision> <!-- Top back beam-->
             <geometry>
-                <box size="0.4 0.15 3.0" />
-            </geometry>
-            <origin rpy="0 0 0" xyz="-0.98 -2.135 0.0" />
+                <box size="0.34 0.15 3.0" />
+            </geometry>
+            <origin rpy="0 0 0" xyz="-1.0 -2.135 0.0" />
         </collision>
         <collision> <!-- Corner Bracket 1-->
@@ -331,4 +356,10 @@
             </geometry>
             <origin rpy="0 0.785 0" xyz="-2.06 -2.135 1.38" />
+        </collision>
+        <collision> <!-- fake floor -->
+            <geometry>
+                <box size="3.0 0.12 3.0" />
+            </geometry>
+            <origin rpy="0 0 0" xyz="-0.65 -0.82 0" />
         </collision>
         <inertial>
@@ -340,6 +371,6 @@
         <parent link="${prefix}robot_stand" />
         <child link="${prefix}base" />
-        <origin rpy="-1.570796 1.570796 0" xyz="-0.148896 -2.047406 0.6277 " />
-<!--        <origin rpy="-1.570796 1.570796 0" xyz="-1.030659 -2.037406 0.7977 " />-->
+<!--        <origin rpy="-1.570796 1.570796 0" xyz="-0.148896 -2.047406 0.6277 " />-->
+        <origin rpy="-1.570796 1.570796 0" xyz="-1.030659 -2.037406 0.7977 " />
         <axis xyz="1 0 0"/>
         <limit effort="1.0" lower="-0.1" upper="1.9" velocity=".01" />
@@ -371,5 +402,30 @@
         <child link="${prefix}camera_link"/>
     </joint>
-    <link name="${prefix}sander_center_link" />
+    <link name="${prefix}sander_center_link" >
+      <visual>
+          <geometry>
+              <cylinder length="0.025" radius="0.06425" />
+          </geometry>
+          <origin rpy="0 0 0" xyz="0 0 0" />
+      </visual>
+      <collision>
+          <geometry>
+              <cylinder length="0.025" radius="0.06425" />
+          </geometry>
+          <origin rpy="0 0 0" xyz="0 0 0" />
+      </collision>
+      <collision>
+          <geometry>
+              <cylinder length="0.03" radius="0.115" />
+          </geometry>
+          <origin rpy="0 0 0" xyz="0 0 -0.105" />
+      </collision>
+<!--      <collision>
+          <geometry>
+              <cylinder length="0.025" radius="0.135" />
+          </geometry>
+          <origin rpy="0 0 0" xyz="0 0 -0.035" />
+      </collision>-->
+    </link>
     <joint name="${prefix}sander_joint" type = "fixed">
         <origin xyz="0.0 -0.15497 0.17503" rpy="0.7854 0.0 0.0"/>

Commit message: Updated flipped EE and cart position

File: crs_support/urdf/crs.urdf.xacro (robot description, xacro)
@@ -223,5 +223,5 @@
     <link name="${prefix}base" />
     <joint name="${prefix}base_link-base_fixed_joint" type="fixed">
-        <origin rpy="0 0 0" xyz="0 0 0" />-->
+        <origin rpy="0 0 3.14" xyz="0 0 0" />-->
         <parent link="${prefix}base" />
         <child link="${prefix}base_link" />
@@ -236,5 +236,5 @@
         <visual>
             <geometry>
-                <mesh filename="package://crs_support/meshes/end_effector/visual/full_ee_v4.stl" />
+                <mesh filename="package://crs_support/meshes/end_effector/visual/flipped_tool.stl" />
             </geometry>
             <material name="Orange">
@@ -242,8 +242,33 @@
             </material>
         </visual>
-        <collision>
-            <geometry>
-                <mesh filename="package://crs_support/meshes/end_effector/collision/full_ee_v4_collision.stl" />
-            </geometry>
+        <visual>
+            <geometry>
+                <mesh filename="package://crs_support/meshes/end_effector/visual/flipped_sander.stl" />
+            </geometry>
+            <material name="Orange">
+                <color rgba="1.0 0.4 0.0 1.0" />
+            </material>
+        </visual>
+        <collision>
+            <geometry>
+                <mesh filename="package://crs_support/meshes/end_effector/collision/flipped_tool_collision.stl" />
+            </geometry>
+        </collision>
+        <collision>
+            <geometry>
+                <mesh filename="package://crs_support/meshes/end_effector/collision/flipped_sander_collision.stl" />
+            </geometry>
+        </collision>
+        <visual>
+          <geometry>
+              <cylinder length="0.05" radius="0.0125" />
+          </geometry>
+          <origin rpy="0 1.57 0" xyz="0.11 -0.055 0.055" />
+        </visual>
+        <collision>
+          <geometry>
+              <cylinder length="0.05" radius="0.0125" />
+          </geometry>
+          <origin rpy="0 1.57 0" xyz="0.11 -0.055 0.055" />
         </collision>
         <inertial>
@@ -269,5 +294,5 @@
         </visual>
         <visual>
-            <origin rpy="1.57079632679 0 0" xyz="0.00 0 -0.1168" />
+            <origin rpy="1.57079632679 0 0" xyz="0.20 0.2 -0.1168" />
             <geometry>
                 <mesh filename="package://crs_support/meshes/Mockup/visual/mockup_cart_v4.stl" />
@@ -278,5 +303,5 @@
         </visual>
         <collision>
-            <origin rpy="1.57079632679 0 0" xyz="0.20 0 -0.1168" />
+            <origin rpy="1.57079632679 0 0" xyz="0.20 0.2 -0.1168" />
             <geometry>
                 <mesh filename="package://crs_support/meshes/Mockup/collision/Mockup3_6_Cart_collision.stl" />
@@ -343,10 +368,10 @@
             <origin rpy="0 0.785 0" xyz="-2.06 -2.135 1.38" />
         </collision>
-        <collision>  fake floor
+        <!--<collision>  fake floor
             <geometry>
                 <box size="3.0 0.12 2.5" />
             </geometry>
             <origin rpy="0 0 0" xyz="-0.65 -0.82 0" />
-        </collision>
+        </collision>-->
         <inertial>
             <mass value="0.1" />
@@ -357,5 +382,5 @@
         <parent link="${prefix}robot_stand" />
         <child link="${prefix}base" />
-        <origin rpy="-1.570796 1.570796 0" xyz="-1.030659 -2.037406 0.7977 " />
+        <origin rpy="-1.570796 -1.570796 0.0" xyz="-1.030659 -2.037406 0.7977 " />
         <axis xyz="1 0 0"/>
         <limit effort="1.0" lower="-0.1" upper="1.9" velocity=".01" />
@@ -389,5 +414,5 @@
       <visual>
           <geometry>
-              <cylinder length="0.025" radius="0.06425" />
+              <cylinder length="0.06" radius="0.06425" />
           </geometry>
           <origin rpy="0 0 0" xyz="0 0 0" />
@@ -399,14 +424,38 @@
           <origin rpy="0 0 0" xyz="0 0 0" />
       </collision>
+      <visual>
+          <geometry>
+              <cylinder length="0.20" radius="0.0125" />
+          </geometry>
+          <origin rpy="1.57 0 0" xyz="-0.0175 -0.1 -.0375" />
+      </visual>
+      <visual>
+          <geometry>
+              <cylinder length="0.0254" radius="0.0125" />
+          </geometry>
+          <origin rpy="0 1.57 0" xyz="0.0 -0.2 -.0375" />
+      </visual>
+      <collision>
+          <geometry>
+              <cylinder length="0.20" radius="0.0125" />
+          </geometry>
+          <origin rpy="1.57 0 0" xyz="-0.0175 -0.1 -.0375" />
+      </collision>
+      <collision>
+          <geometry>
+              <cylinder length="0.0254" radius="0.0125" />
+          </geometry>
+          <origin rpy="0 1.57 0" xyz="0.0 -0.2 -.0375" />
+      </collision>
     </link>
     <joint name="${prefix}sander_intermediate_to_sander_center_link" type="fixed">
       <parent link="${prefix}sander_intermediate_link" />
       <child link="${prefix}sander_center_link" />
-      <origin  xyz="0.0 0.0 0.0125" rpy="0.0 0.0 0.0"/>
+      <origin  xyz="0.0 0.0 0.03" rpy="0.0 0.0 0.0"/>
     </joint>
     <joint name="${prefix}tool0_to_sander_intermediate_link" type="fixed">
         <parent link="${prefix}eoat_link" />
         <child link="${prefix}sander_intermediate_link" />
-        <origin xyz="0.0 -0.15497 0.17503" rpy="0.7854 0.0 0.0"/>
+        <origin xyz="0.0 -0.17503 0.15497" rpy="0.7854 0.0 0.0"/>
     </joint>
     <transmission name="trans_shoulder_pan_joint">

Commit message: Updated mesh names and cleaned up urdfs

File: crs_support/urdf/crs.urdf.xacro (robot description, xacro)
@@ -236,5 +236,5 @@
         <visual>
             <geometry>
-                <mesh filename="package://crs_support/meshes/end_effector/visual/flipped_tool.stl" />
+                <mesh filename="package://crs_support/meshes/end_effector/visual/tool.stl" />
             </geometry>
             <material name="Orange">
@@ -244,5 +244,5 @@
         <visual>
             <geometry>
-                <mesh filename="package://crs_support/meshes/end_effector/visual/flipped_sander.stl" />
+                <mesh filename="package://crs_support/meshes/end_effector/visual/sander.stl" />
             </geometry>
             <material name="Orange">
@@ -252,10 +252,10 @@
         <collision>
             <geometry>
-                <mesh filename="package://crs_support/meshes/end_effector/collision/flipped_tool_collision.stl" />
-            </geometry>
-        </collision>
-        <collision>
-            <geometry>
-                <mesh filename="package://crs_support/meshes/end_effector/collision/flipped_sander_collision.stl" />
+                <mesh filename="package://crs_support/meshes/end_effector/collision/tool_collision.stl" />
+            </geometry>
+        </collision>
+        <collision>
+            <geometry>
+                <mesh filename="package://crs_support/meshes/end_effector/collision/sander_collision.stl" />
             </geometry>
         </collision>

Commit message: Updated collision to account for tool changer stations

File: crs_support/urdf/crs.urdf.xacro (robot description, xacro)
@@ -328,5 +328,5 @@
         <collision> Back Wall bottom Half
             <geometry>
-                <box size="0.1 1.1 3.0" />
+                <box size="0.4 1.1 3.0" />
             </geometry>
             <origin rpy="0 0 0" xyz="-2.06 -0.6 0.0" />

Commit message: Cleaned up some comments

File: crs_support/urdf/crs.urdf.xacro (robot description, xacro)
@@ -314,10 +314,10 @@
             <origin rpy="0 0 0" xyz="-0.5 -1.1 1.38" />
         </collision>
-       <!-- <collision> Left Wall
+        <collision> Left Wall
             <geometry>
                 <box size="3.0 2.14 0.1" />
             </geometry>
             <origin rpy="0 0 0" xyz="-0.5 -1.1 -1.33" />
-        </collision>-->
+        </collision>
         <collision> Front Wall
             <geometry>
@@ -356,10 +356,10 @@
             <origin rpy="0 0 0" xyz="-1.0 -2.135 0.0" />
         </collision>
-        <!--<collision> Corner Bracket 1
+        <collision> Corner Bracket 1
             <geometry>
                 <box size="1.25 0.12 1.25" />
             </geometry>
             <origin rpy="0 0.785 0" xyz="-2.06 -2.135 -1.33" />
-        </collision>-->
+        </collision>
         <collision> Corner Bracket 2
             <geometry>
@@ -382,6 +382,6 @@
         <parent link="${prefix}robot_stand" />
         <child link="${prefix}base" />
-<!--        <origin rpy="-1.570796 -1.570796 0.0" xyz="-1.030659 -2.037406 0.7977 " />-->
-        <origin rpy="-1.570796 -1.570796 0.0" xyz="-1.030659 -2.037406 0.2 " />
+<!--        <origin rpy="-1.570796 -1.570796 0.0" xyz="-1.030659 -2.037406 0.7977 " /> Original position -->
+        <origin rpy="-1.570796 -1.570796 0.0" xyz="-1.030659 -2.037406 0.2 " /> Middle position
         <axis xyz="1 0 0"/>
         <limit effort="1.0" lower="-0.1" upper="1.9" velocity=".01" />

Commit message: Updated base position to match WSU workcell

File: crs_support/urdf/crs.urdf.xacro (robot description, xacro)
@@ -383,5 +383,5 @@
         <child link="${prefix}base" />
 <!--        <origin rpy="-1.570796 -1.570796 0.0" xyz="-1.030659 -2.037406 0.7977 " /> Original position -->
-        <origin rpy="-1.570796 -1.570796 0.0" xyz="-1.030659 -2.037406 0.2 " /> Middle position
+        <origin rpy="-1.570796 -1.570796 0.0" xyz="-1.030659 -2.037406 0.153175 " /> Middle position
         <axis xyz="1 0 0"/>
         <limit effort="1.0" lower="-0.1" upper="1.9" velocity=".01" />

Commit message: initial joint values can now be set for gazebo

File: crs_support/urdf/crs.urdf.xacro (robot description, xacro)
@@ -629,4 +629,8 @@
             </ros>
             <update_rate>20</update_rate>
+            <initial_joint_positions>
+              <joint name="${prefix}shoulder_lift_joint" value="-0.5"/>
+              <joint name="${prefix}elbow_joint" value="0.5"/>
+            </initial_joint_positions>
         </plugin>
     </gazebo>

Commit message: Clang formatting and various integration changes

File: crs_support/urdf/crs.urdf.xacro (robot description, xacro)
@@ -29,5 +29,7 @@
         <origin rpy="0 0 3.14159249728" xyz="0 0 0.180920744391" />
         <axis xyz="0 0 1" />
-        <limit effort="330.0" lower="-4" upper="3.28" velocity="3.14" />
+        <!--limit effort="330.0" lower="-2.6" upper="2.4" velocity="3.14" /-->
+<!--        <limit effort="330.0" lower="-4" upper="3.28" velocity="3.14" />-->
+        <limit effort="330.0" lower="-4.3" upper="4.3" velocity="3.14" />
         <dynamics damping="0.0" friction="0.0" />
     </joint>
@@ -120,4 +122,5 @@
         <axis xyz="0 0 1" />
         <limit effort="54.0" lower="-6.28318530718" upper="6.28318530718" velocity="6.28" />
+ <!--       <limit effort="54.0" lower="-4.2" upper="0.7" velocity="6.28" /-->
         <dynamics damping="0.0" friction="0.0" />
     </joint>
@@ -180,4 +183,5 @@
         <axis xyz="0 0 1" />
         <limit effort="54.0" lower="-6.28318530718" upper="6.28318530718" velocity="6.28" />
+<!--        <limit effort="54.0" lower="-2.6" upper="4.9" velocity="6.28" /-->
         <dynamics damping="0.0" friction="0.0" />
     </joint>
@@ -294,5 +298,7 @@
         </visual>
         <visual>
-            <origin rpy="1.57079632679 0 0" xyz="0.20 0.2 -0.1168" />
+<!--            <origin rpy="1.57079632679 0 0" xyz="0.20 0.2 -0.1168" />-->
+<!--            <origin rpy="1.57079632679 0 0" xyz="0.53 0.2 -0.1168" />-->
+            <origin rpy="1.57079632679 0 0" xyz="0.7 0.2 -0.1168" />
             <geometry>
                 <mesh filename="package://crs_support/meshes/Mockup/visual/mockup_cart_v4.stl" />
@@ -303,12 +309,15 @@
         </visual>
         <collision>
-            <origin rpy="1.57079632679 0 0" xyz="0.20 0.2 -0.1168" />
+            <!--<origin rpy="1.57079632679 0 0" xyz="0.20 0.2 -0.1168" />-->
+<!--            <origin rpy="1.57079632679 0 0" xyz="0.53 0.2 -0.1168" />-->
+            <origin rpy="1.57079632679 0 0" xyz="0.7 0.2 -0.1168" />
             <geometry>
                 <mesh filename="package://crs_support/meshes/Mockup/collision/Mockup3_6_Cart_collision.stl" />
             </geometry>
         </collision>
-        <collision> <!-- Right Wall-->
-            <geometry>
-                <box size="3.0 2.14 0.1" />
+        <collision>  Right Wall
+            <geometry>
+<!--                <box size="3.0 2.14 0.1" />-->
+                <box size="3.0 2.14 0.2" />
             </geometry>
             <origin rpy="0 0 0" xyz="-0.5 -1.1 1.38" />
@@ -316,5 +325,6 @@
         <collision> Left Wall
             <geometry>
-                <box size="3.0 2.14 0.1" />
+<!--                <box size="3.0 2.14 0.1" />-->
+                <box size="3.0 2.14 0.2" />
             </geometry>
             <origin rpy="0 0 0" xyz="-0.5 -1.1 -1.33" />
@@ -322,20 +332,22 @@
         <collision> Front Wall
             <geometry>
+<!--                <box size="0.1 2.14 3.0" />-->
                 <box size="0.1 2.14 3.0" />
             </geometry>
             <origin rpy="0 0 0" xyz="0.85 -1.1 0.0" />
         </collision>
-        <collision> Back Wall bottom Half
-            <geometry>
-                <box size="0.4 1.1 3.0" />
+        <collision> Back Wall bottom Half NOW NO TOOLCHANGERS PRESENT
+            <geometry>
+<!--                <box size="0.4 1.1 3.0" />-->
+                <box size="0.15 3.1 3.0" />
             </geometry>
             <origin rpy="0 0 0" xyz="-2.06 -0.6 0.0" />
         </collision>
-        <collision> Back Wall top beam
+<!--           <collision> Back Wall top beam
             <geometry>
                 <box size="1.25 0.12 3.0" />
             </geometry>
             <origin rpy="0 0 0" xyz="0.38 -2.135 0.0" />
-        </collision>
+        </collision>-->
         <collision> Back Wall Half right
             <geometry>
@@ -350,5 +362,5 @@
             <origin rpy="0.786 0 0" xyz="-2.06 -1.9 -1.15" />
         </collision>
-        <collision> <!-- Top back beam-->
+        <collision> Top back beam
             <geometry>
                 <box size="0.34 0.15 3.0" />
@@ -356,4 +368,18 @@
             <origin rpy="0 0 0" xyz="-1.0 -2.135 0.0" />
         </collision>
+        <!--added by Bharath/Joe on 9/23 to avoid collision-->
+<!--        <collision> Temp block
+            <geometry>
+                <box size="1 1.1 0.1" />
+            </geometry>
+            <origin rpy="0 0.42 0" xyz="-0.0 -0.55 0.7" />
+        </collision>
+        <collision> Temp block2
+            <geometry>
+                <box size="1.5 1.2 0.1" />
+            </geometry>
+            <origin rpy="0 0.42 0" xyz="-0.17 -0.75 -0.9" />
+        </collision>-->
+        <!--added by Bharath/Joe on 9/23 to avoid collision-->
         <collision> Corner Bracket 1
             <geometry>
@@ -367,4 +393,16 @@
             </geometry>
             <origin rpy="0 0.785 0" xyz="-2.06 -2.135 1.38" />
+        </collision>
+        <collision> Corner Bracket 3
+            <geometry>
+                <box size="1.25 0.12 1.25" />
+            </geometry>
+            <origin rpy="0 0.785 0" xyz="0.85 -2.135 -1.33" />
+        </collision>
+        <collision> Corner Bracket 4
+            <geometry>
+                <box size="1.25 0.12 1.25" />
+            </geometry>
+            <origin rpy="0 0.785 0" xyz="0.85 -2.135 1.38" />
         </collision>
         <!--<collision>  fake floor
@@ -448,4 +486,11 @@
           </geometry>
           <origin rpy="0 1.57 0" xyz="0.0 -0.2 -.0375" />
+      </collision>
+<!--Adding collision geom for camera cable-->
+      <collision>
+          <geometry>
+              <cylinder length="0.05" radius="0.0125" />
+          </geometry>
+          <origin rpy="0 1.57 0" xyz="0.075 0.10 -.25" />
       </collision>
     </link>
