Commit message: commiting final WSU changes to test part TRL6 trials

File: crs_support/urdf/crs.urdf.xacro (robot description, xacro)
@@ -294,5 +294,7 @@
         </visual>
         <visual>
-            <origin rpy="1.57079632679 0 0" xyz="0.20 0.2 -0.1168" />
+<!--            <origin rpy="1.57079632679 0 0" xyz="0.20 0.2 -0.1168" />-->
+<!--            <origin rpy="1.57079632679 0 0" xyz="0.53 0.2 -0.1168" />-->
+            <origin rpy="1.57079632679 0.42 0" xyz="0.7 0.2 -0.1168" />
             <geometry>
                 <mesh filename="package://crs_support/meshes/Mockup/visual/mockup_cart_v4.stl" />
@@ -303,12 +305,15 @@
         </visual>
         <collision>
-            <origin rpy="1.57079632679 0 0" xyz="0.20 0.2 -0.1168" />
+            <!--<origin rpy="1.57079632679 0 0" xyz="0.20 0.2 -0.1168" />-->
+<!--            <origin rpy="1.57079632679 0 0" xyz="0.53 0.2 -0.1168" />-->
+            <origin rpy="1.57079632679 0.42 0" xyz="0.7 0.2 -0.1168" />
             <geometry>
                 <mesh filename="package://crs_support/meshes/Mockup/collision/Mockup3_6_Cart_collision.stl" />
             </geometry>
         </collision>
-        <collision> <!-- Right Wall-->
-            <geometry>
-                <box size="3.0 2.14 0.1" />
+        <collision>  Right Wall
+            <geometry>
+<!--                <box size="3.0 2.14 0.1" />-->
+                <box size="3.0 2.14 0.2" />
             </geometry>
             <origin rpy="0 0 0" xyz="-0.5 -1.1 1.38" />
@@ -316,5 +321,6 @@
         <collision> Left Wall
             <geometry>
-                <box size="3.0 2.14 0.1" />
+<!--                <box size="3.0 2.14 0.1" />-->
+                <box size="3.0 2.14 0.2" />
             </geometry>
             <origin rpy="0 0 0" xyz="-0.5 -1.1 -1.33" />
@@ -322,4 +328,5 @@
         <collision> Front Wall
             <geometry>
+<!--                <box size="0.1 2.14 3.0" />-->
                 <box size="0.1 2.14 3.0" />
             </geometry>
@@ -328,14 +335,15 @@
         <collision> Back Wall bottom Half
             <geometry>
-                <box size="0.4 1.1 3.0" />
+<!--                <box size="0.4 1.1 3.0" />-->
+                <box size="0.6 3.1 3.0" />
             </geometry>
             <origin rpy="0 0 0" xyz="-2.06 -0.6 0.0" />
         </collision>
-        <collision> Back Wall top beam
+<!--           <collision> Back Wall top beam
             <geometry>
                 <box size="1.25 0.12 3.0" />
             </geometry>
             <origin rpy="0 0 0" xyz="0.38 -2.135 0.0" />
-        </collision>
+        </collision>-->
         <collision> Back Wall Half right
             <geometry>
@@ -350,5 +358,5 @@
             <origin rpy="0.786 0 0" xyz="-2.06 -1.9 -1.15" />
         </collision>
-        <collision> <!-- Top back beam-->
+        <collision> Top back beam
             <geometry>
                 <box size="0.34 0.15 3.0" />
@@ -356,4 +364,18 @@
             <origin rpy="0 0 0" xyz="-1.0 -2.135 0.0" />
         </collision>
+        <!--added by Bharath/Joe on 9/23 to avoid collision-->
+        <collision> Temp block
+            <geometry>
+                <box size="1 1.1 0.1" />
+            </geometry>
+            <origin rpy="0 0.42 0" xyz="-0.0 -0.55 0.7" />
+        </collision>
+        <collision> Temp block2
+            <geometry>
+                <box size="1.5 1.2 0.1" />
+            </geometry>
+            <origin rpy="0 0.42 0" xyz="-0.17 -0.75 -0.9" />
+        </collision>
+        <!--added by Bharath/Joe on 9/23 to avoid collision-->
         <collision> Corner Bracket 1
             <geometry>
@@ -367,4 +389,16 @@
             </geometry>
             <origin rpy="0 0.785 0" xyz="-2.06 -2.135 1.38" />
+        </collision>
+        <collision> Corner Bracket 3
+            <geometry>
+                <box size="1.25 0.12 1.25" />
+            </geometry>
+            <origin rpy="0 0.785 0" xyz="0.85 -2.135 -1.33" />
+        </collision>
+        <collision> Corner Bracket 4
+            <geometry>
+                <box size="1.25 0.12 1.25" />
+            </geometry>
+            <origin rpy="0 0.785 0" xyz="0.85 -2.135 1.38" />
         </collision>
         <!--<collision>  fake floor
@@ -448,4 +482,11 @@
           </geometry>
           <origin rpy="0 1.57 0" xyz="0.0 -0.2 -.0375" />
+      </collision>
+<!--Adding collision geom for camera cable-->
+      <collision>
+          <geometry>
+              <cylinder length="0.05" radius="0.0125" />
+          </geometry>
+          <origin rpy="0 1.57 0" xyz="0.075 0.10 -.25" />
       </collision>
     </link>

Commit message: End of day before revert to test

File: crs_support/urdf/crs.urdf.xacro (robot description, xacro)
@@ -29,4 +29,5 @@
         <origin rpy="0 0 3.14159249728" xyz="0 0 0.180920744391" />
         <axis xyz="0 0 1" />
+        <!--limit effort="330.0" lower="-2.6" upper="2.4" velocity="3.14" /-->
         <limit effort="330.0" lower="-4" upper="3.28" velocity="3.14" />
         <dynamics damping="0.0" friction="0.0" />
@@ -119,5 +120,6 @@
         <origin rpy="3.13872123266 -3.14053617519 3.14158723656" xyz="-0.571064941288 0.000500820247035 0.174414995927" />
         <axis xyz="0 0 1" />
-        <limit effort="54.0" lower="-6.28318530718" upper="6.28318530718" velocity="6.28" />
+        <limit effort="54.0" lower="-6.28318530718" upper="6.28318530718" velocity="6.28" />>
+ <!--       <limit effort="54.0" lower="-4.2" upper="0.7" velocity="6.28" /-->
         <dynamics damping="0.0" friction="0.0" />
     </joint>
@@ -179,5 +181,6 @@
         <origin rpy="1.57170379674 3.14159265359 3.14159254819" xyz="1.57784168351e-05 0.115533666641 0.000104843358957" />
         <axis xyz="0 0 1" />
-        <limit effort="54.0" lower="-6.28318530718" upper="6.28318530718" velocity="6.28" />
+        <limit effort="54.0" lower="-6.28318530718" upper="6.28318530718" velocity="6.28" />>
+<!--        <limit effort="54.0" lower="-2.6" upper="4.9" velocity="6.28" /-->
         <dynamics damping="0.0" friction="0.0" />
     </joint>
@@ -296,5 +299,5 @@
 <!--            <origin rpy="1.57079632679 0 0" xyz="0.20 0.2 -0.1168" />-->
 <!--            <origin rpy="1.57079632679 0 0" xyz="0.53 0.2 -0.1168" />-->
-            <origin rpy="1.57079632679 0.42 0" xyz="0.7 0.2 -0.1168" />
+            <origin rpy="1.57079632679 0 0" xyz="0.7 0.2 -0.1168" />
             <geometry>
                 <mesh filename="package://crs_support/meshes/Mockup/visual/mockup_cart_v4.stl" />
@@ -307,5 +310,5 @@
             <!--<origin rpy="1.57079632679 0 0" xyz="0.20 0.2 -0.1168" />-->
 <!--            <origin rpy="1.57079632679 0 0" xyz="0.53 0.2 -0.1168" />-->
-            <origin rpy="1.57079632679 0.42 0" xyz="0.7 0.2 -0.1168" />
+            <origin rpy="1.57079632679 0 0" xyz="0.7 0.2 -0.1168" />
             <geometry>
                 <mesh filename="package://crs_support/meshes/Mockup/collision/Mockup3_6_Cart_collision.stl" />
@@ -333,8 +336,8 @@
             <origin rpy="0 0 0" xyz="0.85 -1.1 0.0" />
         </collision>
-        <collision> Back Wall bottom Half
+        <collision> Back Wall bottom Half NOW NO TOOLCHANGERS PRESENT
             <geometry>
 <!--                <box size="0.4 1.1 3.0" />-->
-                <box size="0.6 3.1 3.0" />
+                <box size="0.15 3.1 3.0" />
             </geometry>
             <origin rpy="0 0 0" xyz="-2.06 -0.6 0.0" />
@@ -365,5 +368,5 @@
         </collision>
         <!--added by Bharath/Joe on 9/23 to avoid collision-->
-        <collision> Temp block
+<!--        <collision> Temp block
             <geometry>
                 <box size="1 1.1 0.1" />
@@ -376,5 +379,5 @@
             </geometry>
             <origin rpy="0 0.42 0" xyz="-0.17 -0.75 -0.9" />
-        </collision>
+        </collision>-->
         <!--added by Bharath/Joe on 9/23 to avoid collision-->
         <collision> Corner Bracket 1

Commit message: Branch to save TRL-6 part 35 status

File: crs_support/urdf/crs.urdf.xacro (robot description, xacro)
@@ -30,5 +30,6 @@
         <axis xyz="0 0 1" />
         <!--limit effort="330.0" lower="-2.6" upper="2.4" velocity="3.14" /-->
-        <limit effort="330.0" lower="-4" upper="3.28" velocity="3.14" />
+<!--        <limit effort="330.0" lower="-4" upper="3.28" velocity="3.14" />-->
+        <limit effort="330.0" lower="-4.3" upper="4.3" velocity="3.14" />
         <dynamics damping="0.0" friction="0.0" />
     </joint>
@@ -120,5 +121,5 @@
         <origin rpy="3.13872123266 -3.14053617519 3.14158723656" xyz="-0.571064941288 0.000500820247035 0.174414995927" />
         <axis xyz="0 0 1" />
-        <limit effort="54.0" lower="-6.28318530718" upper="6.28318530718" velocity="6.28" />>
+        <limit effort="54.0" lower="-6.28318530718" upper="6.28318530718" velocity="6.28" />
  <!--       <limit effort="54.0" lower="-4.2" upper="0.7" velocity="6.28" /-->
         <dynamics damping="0.0" friction="0.0" />
@@ -181,5 +182,5 @@
         <origin rpy="1.57170379674 3.14159265359 3.14159254819" xyz="1.57784168351e-05 0.115533666641 0.000104843358957" />
         <axis xyz="0 0 1" />
-        <limit effort="54.0" lower="-6.28318530718" upper="6.28318530718" velocity="6.28" />>
+        <limit effort="54.0" lower="-6.28318530718" upper="6.28318530718" velocity="6.28" />
 <!--        <limit effort="54.0" lower="-2.6" upper="4.9" velocity="6.28" /-->
         <dynamics damping="0.0" friction="0.0" />

Commit message: restores robot base location, scan poses are now reachable

File: crs_support/urdf/crs.urdf.xacro (robot description, xacro)
@@ -29,7 +29,5 @@
         <origin rpy="0 0 3.14159249728" xyz="0 0 0.180920744391" />
         <axis xyz="0 0 1" />
-        <!--limit effort="330.0" lower="-2.6" upper="2.4" velocity="3.14" /-->
-<!--        <limit effort="330.0" lower="-4" upper="3.28" velocity="3.14" />-->
-        <limit effort="330.0" lower="-4.3" upper="4.3" velocity="3.14" />
+        <limit effort="330.0" lower="-4" upper="3.28" velocity="3.14" />
         <dynamics damping="0.0" friction="0.0" />
     </joint>
@@ -122,5 +120,4 @@
         <axis xyz="0 0 1" />
         <limit effort="54.0" lower="-6.28318530718" upper="6.28318530718" velocity="6.28" />
- <!--       <limit effort="54.0" lower="-4.2" upper="0.7" velocity="6.28" /-->
         <dynamics damping="0.0" friction="0.0" />
     </joint>
@@ -183,5 +180,4 @@
         <axis xyz="0 0 1" />
         <limit effort="54.0" lower="-6.28318530718" upper="6.28318530718" velocity="6.28" />
-<!--        <limit effort="54.0" lower="-2.6" upper="4.9" velocity="6.28" /-->
         <dynamics damping="0.0" friction="0.0" />
     </joint>
@@ -298,7 +294,5 @@
         </visual>
         <visual>
-<!--            <origin rpy="1.57079632679 0 0" xyz="0.20 0.2 -0.1168" />-->
-<!--            <origin rpy="1.57079632679 0 0" xyz="0.53 0.2 -0.1168" />-->
-            <origin rpy="1.57079632679 0 0" xyz="0.7 0.2 -0.1168" />
+            <origin rpy="1.57079632679 0 0" xyz="0.20 0.2 -0.1168" />
             <geometry>
                 <mesh filename="package://crs_support/meshes/Mockup/visual/mockup_cart_v4.stl" />
@@ -309,22 +303,18 @@
         </visual>
         <collision>
-            <!--<origin rpy="1.57079632679 0 0" xyz="0.20 0.2 -0.1168" />-->
-<!--            <origin rpy="1.57079632679 0 0" xyz="0.53 0.2 -0.1168" />-->
-            <origin rpy="1.57079632679 0 0" xyz="0.7 0.2 -0.1168" />
+            <origin rpy="1.57079632679 0 0" xyz="0.20 0.2 -0.1168" />
             <geometry>
                 <mesh filename="package://crs_support/meshes/Mockup/collision/Mockup3_6_Cart_collision.stl" />
             </geometry>
         </collision>
-        <collision>  Right Wall
-            <geometry>
-<!--                <box size="3.0 2.14 0.1" />-->
-                <box size="3.0 2.14 0.2" />
+        <collision> <!-- Right Wall-->
+            <geometry>
+                <box size="3.0 2.14 0.1" />
             </geometry>
             <origin rpy="0 0 0" xyz="-0.5 -1.1 1.38" />
         </collision>
-        <collision> Left Wall
-            <geometry>
-<!--                <box size="3.0 2.14 0.1" />-->
-                <box size="3.0 2.14 0.2" />
+        <collision> <!-- Left Wall-->
+            <geometry>
+                <box size="3.0 2.14 0.1" />
             </geometry>
             <origin rpy="0 0 0" xyz="-0.5 -1.1 -1.33" />
@@ -332,22 +322,20 @@
         <collision> Front Wall
             <geometry>
-<!--                <box size="0.1 2.14 3.0" />-->
                 <box size="0.1 2.14 3.0" />
             </geometry>
             <origin rpy="0 0 0" xyz="0.85 -1.1 0.0" />
         </collision>
-        <collision> Back Wall bottom Half NOW NO TOOLCHANGERS PRESENT
-            <geometry>
-<!--                <box size="0.4 1.1 3.0" />-->
-                <box size="0.15 3.1 3.0" />
+        <collision> Back Wall bottom Half
+            <geometry>
+                <box size="0.4 1.1 3.0" />
             </geometry>
             <origin rpy="0 0 0" xyz="-2.06 -0.6 0.0" />
         </collision>
-<!--           <collision> Back Wall top beam
+        <collision> Back Wall top beam
             <geometry>
                 <box size="1.25 0.12 3.0" />
             </geometry>
             <origin rpy="0 0 0" xyz="0.38 -2.135 0.0" />
-        </collision>-->
+        </collision>
         <collision> Back Wall Half right
             <geometry>
@@ -362,5 +350,5 @@
             <origin rpy="0.786 0 0" xyz="-2.06 -1.9 -1.15" />
         </collision>
-        <collision> Top back beam
+        <collision> <!-- Top back beam-->
             <geometry>
                 <box size="0.34 0.15 3.0" />
@@ -368,19 +356,5 @@
             <origin rpy="0 0 0" xyz="-1.0 -2.135 0.0" />
         </collision>
-        <!--added by Bharath/Joe on 9/23 to avoid collision-->
-<!--        <collision> Temp block
-            <geometry>
-                <box size="1 1.1 0.1" />
-            </geometry>
-            <origin rpy="0 0.42 0" xyz="-0.0 -0.55 0.7" />
-        </collision>
-        <collision> Temp block2
-            <geometry>
-                <box size="1.5 1.2 0.1" />
-            </geometry>
-            <origin rpy="0 0.42 0" xyz="-0.17 -0.75 -0.9" />
-        </collision>-->
-        <!--added by Bharath/Joe on 9/23 to avoid collision-->
-        <collision> Corner Bracket 1
+        <collision> <!-- Corner Bracket 1-->
             <geometry>
                 <box size="1.25 0.12 1.25" />
@@ -388,21 +362,9 @@
             <origin rpy="0 0.785 0" xyz="-2.06 -2.135 -1.33" />
         </collision>
-        <collision> Corner Bracket 2
+        <collision> <!-- Corner Bracket 2-->
             <geometry>
                 <box size="1.25 0.12 1.25" />
             </geometry>
             <origin rpy="0 0.785 0" xyz="-2.06 -2.135 1.38" />
-        </collision>
-        <collision> Corner Bracket 3
-            <geometry>
-                <box size="1.25 0.12 1.25" />
-            </geometry>
-            <origin rpy="0 0.785 0" xyz="0.85 -2.135 -1.33" />
-        </collision>
-        <collision> Corner Bracket 4
-            <geometry>
-                <box size="1.25 0.12 1.25" />
-            </geometry>
-            <origin rpy="0 0.785 0" xyz="0.85 -2.135 1.38" />
         </collision>
         <!--<collision>  fake floor
@@ -420,6 +382,5 @@
         <parent link="${prefix}robot_stand" />
         <child link="${prefix}base" />
-<!--        <origin rpy="-1.570796 -1.570796 0.0" xyz="-1.030659 -2.037406 0.7977 " /> Original position -->
-        <origin rpy="-1.570796 -1.570796 0.0" xyz="-1.030659 -2.037406 0.153175 " /> Middle position
+        <origin rpy="-1.570796 -1.570796 0.0" xyz="-1.030659 -2.037406 0.7977 " />
         <axis xyz="1 0 0"/>
         <limit effort="1.0" lower="-0.1" upper="1.9" velocity=".01" />
@@ -486,11 +447,4 @@
           </geometry>
           <origin rpy="0 1.57 0" xyz="0.0 -0.2 -.0375" />
-      </collision>
-<!--Adding collision geom for camera cable-->
-      <collision>
-          <geometry>
-              <cylinder length="0.05" radius="0.0125" />
-          </geometry>
-          <origin rpy="0 1.57 0" xyz="0.075 0.10 -.25" />
       </collision>
     </link>
@@ -674,8 +628,4 @@
             </ros>
             <update_rate>20</update_rate>
-            <initial_joint_positions>
-              <joint name="${prefix}shoulder_lift_joint" value="-0.5"/>
-              <joint name="${prefix}elbow_joint" value="0.5"/>
-            </initial_joint_positions>
         </plugin>
     </gazebo>
